File: 65c816/65c816board/65c816board.sch (KiCad schematic (older format))
At the start: 4 parts, among them U1 w65c816, U2 74HC573, U3 74HC32, U4 74HC04

Commit message: Breadboard layout for the 65C816 CPU board.
Parts:
- added C1, C2, C3, C4: 100nF, symbol Device:C_Small
- added J?: Conn_01x34_Male, symbol Connector:Conn_01x34_Male
- added R1: 1k, symbol Device:R_Small
Connections:
- net labels added: 5V, A0, A1, A10, A11, A12, A13, A14, A15, A16, A17, A18, A2, A3, A4, A5, A6, A7, A8, A9, CLK, D0, D1, D2, D3, D4, D5, D6, D7, GND, RAM, RD, RES, WR
- wire segments 0 -> 186
- no-connect marks 0 -> 11

Commit message: Rework schematics and documentation
Parts:
- C1, C2, C3, C4: footprint (none) -> Capacitor_THT:C_Disc_D3.8mm_W2.6mm_P2.50mm
- J1: renamed from J?; footprint (none) -> Connector_PinHeader_2.54mm:PinHeader_1x34_P2.54mm_Vertical
- R1: footprint (none) -> Resistor_THT:R_Axial_DIN0207_L6.3mm_D2.5mm_P7.62mm_Horizontal
- U1: footprint (none) -> Package_DIP:DIP-40_W15.24mm_Socket
- U2: footprint (none) -> Package_DIP:DIP-20_W7.62mm_Socket
- U3, U4: footprint (none) -> Package_DIP:DIP-14_W7.62mm_Socket
Connections:
- wire segments 186 -> 187
Changed lines of the file:
@@
 F 0 "U3" H 6600 3150 50  0000 R CNN
 F 1 "74HC32" V 6550 2900 50  0000 R CNN
-F 2 "" H 6550 3150 50  0001 C CNN
+F 2 "Package_DIP:DIP-14_W7.62mm_Socket" H 6550 3150 50  0001 C CNN
 F 3 "" H 6550 3150 50  0001 C CNN
 	1    6550 3150
@@
 F 0 "U4" H 7750 3150 50  0000 R CNN
 F 1 "74HC04" V 7700 2900 50  0000 R CNN
-F 2 "" H 7700 3150 50  0001 C CNN
+F 2 "Package_DIP:DIP-14_W7.62mm_Socket" H 7700 3150 50  0001 C CNN
 F 3 "" H 7700 3150 50  0001 C CNN
 	1    7700 3150
@@
 F 0 "U2" H 6000 2050 50  0000 L CNN
 F 1 "74HC573" V 6050 2450 50  0000 L CNN
-F 2 "" H 6050 3150 50  0001 C CNN
+F 2 "Package_DIP:DIP-20_W7.62mm_Socket" H 6050 3150 50  0001 C CNN
 F 3 "" H 6050 3150 50  0001 C CNN
 	1    6050 3150
@@
 	4550 1800 4550 2800
 $Comp
-L Connector:Conn_01x34_Male J?
+L Connector:Conn_01x34_Male J1
 U 1 1 5EE68390
 P 4450 4950
-F 0 "J?" V 4378 4876 50  0000 C CNN
+F 0 "J1" V 4378 4876 50  0000 C CNN
 F 1 "Conn_01x34_Male" V 4287 4876 50  0000 C CNN
-F 2 "" H 4450 4950 50  0001 C CNN
+F 2 "Connector_PinHeader_2.54mm:PinHeader_1x34_P2.54mm_Vertical" H 4450 4950 50  0001 C CNN
 F 3 "~" H 4450 4950 50  0001 C CNN
 	1    4450 4950
@@
 	2400 4200 4900 4200
 $Comp
-L power:PWR_FLAG #FLG?
+L power:PWR_FLAG #FLG0101
 U 1 1 5EE7271F
 P 2400 4100
-F 0 "#FLG?" H 2400 4175 50  0001 C CNN
+F 0 "#FLG0101" H 2400 4175 50  0001 C CNN
 F 1 "PWR_FLAG" V 2400 4228 50  0000 L CNN
 F 2 "" H 2400 4100 50  0001 C CNN
@@
 $EndComp
 $Comp
-L power:PWR_FLAG #FLG?
+L power:PWR_FLAG #FLG0102
 U 1 1 5EE7275A
 P 2400 4200
-F 0 "#FLG?" H 2400 4275 50  0001 C CNN
+F 0 "#FLG0102" H 2400 4275 50  0001 C CNN
 F 1 "PWR_FLAG" V 2400 4328 50  0000 L CNN
 F 2 "" H 2400 4200 50  0001 C CNN
@@
 F 0 "C1" V 4850 3000 50  0000 L CNN
 F 1 "100nF" V 4850 3200 50  0000 L CNN
-F 2 "" H 4800 3150 50  0001 C CNN
+F 2 "Capacitor_THT:C_Disc_D3.8mm_W2.6mm_P2.50mm" H 4800 3150 50  0001 C CNN
 F 3 "~" H 4800 3150 50  0001 C CNN
 	1    4800 3150
@@
 F 0 "C2" V 6150 3000 50  0000 L CNN
 F 1 "100nF" V 6150 3200 50  0000 L CNN
-F 2 "" H 6100 3150 50  0001 C CNN
+F 2 "Capacitor_THT:C_Disc_D3.8mm_W2.6mm_P2.50mm" H 6100 3150 50  0001 C CNN
 F 3 "~" H 6100 3150 50  0001 C CNN
 	1    6100 3150
@@
 F 0 "C3" V 7450 3000 50  0000 L CNN
 F 1 "100nF" V 7450 3200 50  0000 L CNN
-F 2 "" H 7400 3150 50  0001 C CNN
+F 2 "Capacitor_THT:C_Disc_D3.8mm_W2.6mm_P2.50mm" H 7400 3150 50  0001 C CNN
 F 3 "~" H 7400 3150 50  0001 C CNN
 	1    7400 3150
@@
 F 0 "C4" V 8600 3000 50  0000 L CNN
 F 1 "100nF" V 8600 3200 50  0000 L CNN
-F 2 "" H 8550 3150 50  0001 C CNN
+F 2 "Capacitor_THT:C_Disc_D3.8mm_W2.6mm_P2.50mm" H 8550 3150 50  0001 C CNN
 F 3 "~" H 8550 3150 50  0001 C CNN
 	1    8550 3150
@@
 F 0 "U1" H 2800 3200 50  0000 R CNN
 F 1 "w65c816" V 2700 2150 50  0000 R CNN
-F 2 "" H 2700 3150 50  0001 C CNN
+F 2 "Package_DIP:DIP-40_W15.24mm_Socket" H 2700 3150 50  0001 C CNN
 F 3 "" H 2700 3150 50  0001 C CNN
 	1    2700 3150
@@
 F 0 "R1" V 2900 3550 50  0000 L CNN
 F 1 "1k" V 2900 3850 50  0000 L CNN
-F 2 "" H 2850 3750 50  0001 C CNN
+F 2 "Resistor_THT:R_Axial_DIN0207_L6.3mm_D2.5mm_P7.62mm_Horizontal" H 2850 3750 50  0001 C CNN
 F 3 "~" H 2850 3750 50  0001 C CNN
 	1    2850 3750
@@
 Wire Wire Line
 	5250 3500 5250 4750
-Wire Wire Line
-	5350 3500 5350 4750
 Wire Wire Line
 	5450 3500 5450 4750
@@
 	7800 3700 7800 3500
 Wire Wire Line
-	5850 3700 5050 3700
-Wire Wire Line
-	5050 3700 5050 3500
-Connection ~ 5850 3700
-Wire Wire Line
 	6450 2450 8200 2450
 Wire Wire Line
@@
 Wire Wire Line
 	7150 2050 7150 2800
+Wire Wire Line
+	8100 3550 8100 3650
+Wire Wire Line
+	8100 3650 5050 3650
+Connection ~ 8100 3550
+Wire Wire Line
+	5050 3650 5050 3500
+Wire Wire Line
+	5350 3500 5350 4750
 $EndSCHEMATC

Commit message: Working setup for the 65c816
Connections:
- wire segments 187 -> 186
Changed lines of the file:
@@
 	3950 2800 3950 1800
-Wire Wire Line
-	4050 2800 4050 2050
-Wire Wire Line
-	4150 2800 4150 2100
 Wire Wire Line
 	4350 2800 4350 1800
@@
 A15
 Wire Wire Line
-	4250 1800 4250 2150
-Wire Wire Line
 	4050 3500 4050 4750
 Wire Wire Line
@@
 RAM
 Wire Wire Line
-	2400 4100 2500 4100
+	2400 4100 2450 4100
 Wire Wire Line
 	2400 4200 4900 4200
@@
 Connection ~ 8550 2750
 Wire Wire Line
-	2500 4100 2500 2650
-Wire Wire Line
-	2500 2650 3150 2650
+	2450 4100 2450 2650
+Wire Wire Line
+	2450 2650 3150 2650
 Wire Wire Line
 	3150 2650 3150 2800
-Connection ~ 2500 4100
-Wire Wire Line
-	2500 4100 2850 4100
+Connection ~ 2450 4100
+Wire Wire Line
+	2450 4100 2850 4100
 Wire Wire Line
 	2950 3500 2950 4100
@@
 Wire Wire Line
 	2950 4100 3050 4100
-NoConn ~ 3250 2800
 Wire Wire Line
 	3050 3500 3050 4100
@@
 	8200 3550 8200 3500
 Wire Wire Line
-	8800 2300 3050 2300
-Wire Wire Line
-	3050 2300 3050 2800
-Wire Wire Line
 	5850 3700 6750 3700
 Wire Wire Line
@@
 	7800 3700 7800 3500
 Wire Wire Line
-	6450 2450 8200 2450
-Wire Wire Line
 	8100 2800 8100 2400
 Wire Wire Line
@@
 	8300 2750 7800 2750
 Wire Wire Line
-	6950 2800 6950 2550
-Wire Wire Line
-	6950 2550 7900 2550
-Wire Wire Line
-	7900 2550 7900 2800
-Wire Wire Line
 	8000 2800 8000 2600
 Wire Wire Line
-	6750 2800 6750 2150
-Wire Wire Line
-	6750 2150 4250 2150
-Connection ~ 4250 2150
-Wire Wire Line
-	4250 2150 4250 2800
-Wire Wire Line
-	6850 2800 6850 2100
-Wire Wire Line
-	6850 2100 4150 2100
-Connection ~ 4150 2100
-Wire Wire Line
-	4150 2100 4150 1800
-Wire Wire Line
-	7050 2800 7050 2600
-Connection ~ 4050 2050
-Wire Wire Line
-	4050 2050 4050 1800
-Wire Wire Line
-	7250 2800 7250 2700
-Wire Wire Line
-	5450 2700 5450 2800
-Wire Wire Line
 	5750 4000 2600 4000
 Wire Wire Line
@@
 	2600 2750 2600 4000
 Wire Wire Line
-	7250 2700 5450 2700
-Wire Wire Line
 	6650 2800 6650 2750
-Wire Wire Line
-	6650 2750 7400 2750
 Wire Wire Line
 	7400 2750 7500 2750
@@
 Wire Wire Line
 	7500 4100 8650 4100
-Wire Wire Line
-	8000 2600 7150 2600
 Connection ~ 8550 4200
 Wire Wire Line
@@
 	8650 4100 8800 4100
 Wire Wire Line
-	8300 3500 8300 3700
-Wire Wire Line
-	8300 3700 8800 3700
-Wire Wire Line
-	8800 2300 8800 3700
-Wire Wire Line
-	7150 2600 7050 2600
-Wire Wire Line
-	4050 2050 7150 2050
-Wire Wire Line
-	7150 2050 7150 2800
-Wire Wire Line
 	8100 3550 8100 3650
 Wire Wire Line
@@
 Wire Wire Line
 	5350 3500 5350 4750
+Wire Wire Line
+	4250 1800 4250 2800
+Wire Wire Line
+	4150 1800 4150 2100
+Wire Wire Line
+	4050 1800 4050 2800
+Wire Wire Line
+	6450 2450 8200 2450
+Wire Wire Line
+	3250 2800 3250 2050
+Wire Wire Line
+	3250 2050 6850 2050
+Connection ~ 4150 2100
+Wire Wire Line
+	4150 2100 4150 2800
+Wire Wire Line
+	7900 2650 7900 2800
+Wire Wire Line
+	8000 2600 5450 2600
+Wire Wire Line
+	5450 2600 5450 2800
+Wire Wire Line
+	6850 2750 7050 2750
+Wire Wire Line
+	3050 2700 2550 2700
+Wire Wire Line
+	2550 2700 2550 4050
+Wire Wire Line
+	2550 4050 8300 4050
+Wire Wire Line
+	3050 2700 3050 2800
+Wire Wire Line
+	8300 3500 8300 4050
+Wire Wire Line
+	6650 2750 6750 2750
+Wire Wire Line
+	6750 2750 6850 2750
+Wire Wire Line
+	6750 2100 4150 2100
+Wire Wire Line
+	6750 2100 6750 2800
+Wire Wire Line
+	6850 2050 6850 2800
+Wire Wire Line
+	6950 2800 6950 2650
+Wire Wire Line
+	6950 2650 7900 2650
+Wire Wire Line
+	7050 2750 7050 2800
+Connection ~ 7050 2750
+Wire Wire Line
+	7050 2750 7150 2750
+Wire Wire Line
+	7150 2750 7150 2800
+Connection ~ 7150 2750
+Wire Wire Line
+	7150 2750 7400 2750
+NoConn ~ 7250 2800
 $EndSCHEMATC

Commit message: Remove unnecessary pullup at Rdy pin
Parts:
- removed R1: 1k, Resistor_THT:R_Axial_DIN0207_L6.3mm_D2.5mm_P7.62mm_Horizontal, symbol Device:R_Small
Connections:
- wire segments 186 -> 183
- no-connect marks 11 -> 12
Changed lines of the file:
@@
 Connection ~ 2450 4100
-Wire Wire Line
-	2450 4100 2850 4100
 Wire Wire Line
 	2950 3500 2950 4100
@@
 Wire Wire Line
 	3250 4100 4800 4100
-$Comp
-L Device:R_Small R1
-U 1 1 5EE9C159
-P 2850 3750
-F 0 "R1" V 2900 3550 50  0000 L CNN
-F 1 "1k" V 2900 3850 50  0000 L CNN
-F 2 "Resistor_THT:R_Axial_DIN0207_L6.3mm_D2.5mm_P7.62mm_Horizontal" H 2850 3750 50  0001 C CNN
-F 3 "~" H 2850 3750 50  0001 C CNN
-	1    2850 3750
-	1    0    0    -1
-$EndComp
-Wire Wire Line
-	2850 3500 2850 3650
-Wire Wire Line
-	2850 3850 2850 4100
-Connection ~ 2850 4100
-Wire Wire Line
-	2850 4100 2950 4100
 NoConn ~ 2850 2800
 NoConn ~ 3350 3500
@@
 	7150 2750 7400 2750
 NoConn ~ 7250 2800
+Wire Wire Line
+	2450 4100 2950 4100
+NoConn ~ 2850 3500
 $EndSCHEMATC

Commit message: Switch meaning of the A19 pin from RAM to ROM. Use pull-ups instead of pull-downs for the input port.
Parts:
- removed U4: 74HC04, Package_DIP:DIP-14_W7.62mm_Socket, symbol customparts:74HC04
- added U3: 74AC00, symbol customparts:74HC00
- U2: value 74HC573 -> 74AC573
- U4: renamed from U3; value 74HC32 -> 74AC32
Connections:
- net labels added: RD#, RES#, ROM, WR#
- net labels removed: RAM, RD, RES, WR
- wire segments 183 -> 188
- no-connect marks 12 -> 10
Changed lines of the file:
@@
 $EndDescr
 $Comp
-L customparts:74HC32 U3
+L customparts:74HC32 U4
 U 1 1 5EE4132A
-P 6550 3150
-F 0 "U3" H 6600 3150 50  0000 R CNN
-F 1 "74HC32" V 6550 2900 50  0000 R CNN
-F 2 "Package_DIP:DIP-14_W7.62mm_Socket" H 6550 3150 50  0001 C CNN
-F 3 "" H 6550 3150 50  0001 C CNN
-	1    6550 3150
-	0    -1   -1   0
-$EndComp
-$Comp
-L customparts:74HC04 U4
-U 1 1 5EE41390
 P 7700 3150
 F 0 "U4" H 7750 3150 50  0000 R CNN
-F 1 "74HC04" V 7700 2900 50  0000 R CNN
+F 1 "74AC32" V 7700 2900 50  0000 R CNN
 F 2 "Package_DIP:DIP-14_W7.62mm_Socket" H 7700 3150 50  0001 C CNN
 F 3 "" H 7700 3150 50  0001 C CNN
@@
 P 6050 3150
 F 0 "U2" H 6000 2050 50  0000 L CNN
-F 1 "74HC573" V 6050 2450 50  0000 L CNN
+F 1 "74AC573" V 6050 2450 50  0000 L CNN
 F 2 "Package_DIP:DIP-20_W7.62mm_Socket" H 6050 3150 50  0001 C CNN
 F 3 "" H 6050 3150 50  0001 C CNN
@@
 A18
 Text Label 5450 4700 1    50   ~ 0
-RAM
+ROM
 Wire Wire Line
 	2400 4100 2450 4100
@@
 	8550 3050 8550 2750
 Wire Wire Line
-	8550 2750 8300 2750
-Wire Wire Line
 	7800 2750 7800 2800
 Wire Wire Line
@@
 	3750 1800 3750 2800
 Text Label 5550 4700 1    50   ~ 0
-RD
+RD#
 Text Label 5650 4700 1    50   ~ 0
-WR
+WR#
 Text Label 5750 4700 1    50   ~ 0
-RES
+RES#
 Text Label 5850 4700 1    50   ~ 0
 CLK
@@
 	3350 2800 3350 2400
 Wire Wire Line
-	3350 2400 6400 2400
-Wire Wire Line
 	5550 3800 6850 3800
 Wire Wire Line
@@
 	6650 3550 6450 3550
 Wire Wire Line
-	6450 3550 6450 2450
-Wire Wire Line
-	6400 2400 6400 3600
-Connection ~ 6400 2400
-Wire Wire Line
 	7900 3500 7900 3550
-Wire Wire Line
-	7900 3550 8000 3550
 Wire Wire Line
 	8000 3550 8000 3500
@@
 	6750 3700 6750 3500
 Wire Wire Line
-	7800 3700 7800 3500
-Wire Wire Line
-	8100 2800 8100 2400
-Wire Wire Line
-	6400 2400 8100 2400
-Wire Wire Line
-	8200 2450 8200 2800
-NoConn ~ 8400 2800
-Wire Wire Line
-	8300 2800 8300 2750
-Connection ~ 8300 2750
-Wire Wire Line
-	8300 2750 7800 2750
-Wire Wire Line
-	8000 2800 8000 2600
+	7800 3700 7800 3550
+Wire Wire Line
+	8100 2800 8100 2600
 Wire Wire Line
 	5750 4000 2600 4000
@@
 	8650 4100 8800 4100
 Wire Wire Line
-	8100 3550 8100 3650
-Wire Wire Line
-	8100 3650 5050 3650
-Connection ~ 8100 3550
-Wire Wire Line
-	5050 3650 5050 3500
-Wire Wire Line
 	5350 3500 5350 4750
 Wire Wire Line
 	4250 1800 4250 2800
 Wire Wire Line
-	4150 1800 4150 2100
-Wire Wire Line
 	4050 1800 4050 2800
 Wire Wire Line
-	6450 2450 8200 2450
-Wire Wire Line
 	3250 2800 3250 2050
 Wire Wire Line
-	3250 2050 6850 2050
-Connection ~ 4150 2100
-Wire Wire Line
-	4150 2100 4150 2800
-Wire Wire Line
-	7900 2650 7900 2800
-Wire Wire Line
-	8000 2600 5450 2600
-Wire Wire Line
 	5450 2600 5450 2800
 Wire Wire Line
-	6850 2750 7050 2750
-Wire Wire Line
-	3050 2700 2550 2700
-Wire Wire Line
-	2550 2700 2550 4050
-Wire Wire Line
-	2550 4050 8300 4050
-Wire Wire Line
-	3050 2700 3050 2800
-Wire Wire Line
-	8300 3500 8300 4050
-Wire Wire Line
-	6650 2750 6750 2750
-Wire Wire Line
-	6750 2750 6850 2750
-Wire Wire Line
-	6750 2100 4150 2100
-Wire Wire Line
-	6750 2100 6750 2800
-Wire Wire Line
-	6850 2050 6850 2800
+	8300 3500 8300 3650
 Wire Wire Line
 	6950 2800 6950 2650
-Wire Wire Line
-	6950 2650 7900 2650
-Wire Wire Line
-	7050 2750 7050 2800
-Connection ~ 7050 2750
-Wire Wire Line
-	7050 2750 7150 2750
-Wire Wire Line
-	7150 2750 7150 2800
-Connection ~ 7150 2750
-Wire Wire Line
-	7150 2750 7400 2750
-NoConn ~ 7250 2800
 Wire Wire Line
 	2450 4100 2950 4100
 NoConn ~ 2850 3500
+$Comp
+L customparts:74HC00 U3
+U 1 1 5EF3F1D0
+P 6550 3150
+F 0 "U3" H 6650 3150 50  0000 R CNN
+F 1 "74AC00" V 6550 2900 50  0000 R CNN
+F 2 "" H 6550 3150 50  0001 C CNN
+F 3 "" H 6550 3150 50  0001 C CNN
+	1    6550 3150
+	0    -1   -1   0
+$EndComp
+Wire Wire Line
+	6650 2750 7400 2750
+Wire Wire Line
+	5450 2600 8100 2600
+Wire Wire Line
+	8000 2050 8000 2800
+Wire Wire Line
+	3250 2050 8000 2050
+Wire Wire Line
+	4150 2150 7900 2150
+Connection ~ 4150 2150
+Wire Wire Line
+	4150 2150 4150 2800
+Wire Wire Line
+	7900 2150 7900 2800
+Wire Wire Line
+	4150 1800 4150 2150
+Wire Wire Line
+	6450 2400 6450 3550
+Wire Wire Line
+	3350 2400 6450 2400
+Wire Wire Line
+	6450 2400 6750 2400
+Wire Wire Line
+	6750 2400 6750 2800
+Connection ~ 6450 2400
+Wire Wire Line
+	6750 2400 6850 2400
+Wire Wire Line
+	6850 2400 6850 2800
+Connection ~ 6750 2400
+Wire Wire Line
+	6950 2650 6400 2650
+Wire Wire Line
+	6400 2650 6400 3600
+Wire Wire Line
+	7800 3550 7900 3550
+Connection ~ 7800 3550
+Wire Wire Line
+	7800 3550 7800 3500
+Wire Wire Line
+	8000 3550 8100 3550
+Connection ~ 8100 3550
+Wire Wire Line
+	7150 2650 7150 2800
+Wire Wire Line
+	7050 2800 7050 2650
+Wire Wire Line
+	7050 2650 7150 2650
+Wire Wire Line
+	8300 3650 8800 3650
+Wire Wire Line
+	8800 3650 8800 2600
+Wire Wire Line
+	8800 2600 8300 2600
+Wire Wire Line
+	8200 2600 8200 2650
+Wire Wire Line
+	7800 2750 8550 2750
+Wire Wire Line
+	8300 2600 8300 2800
+Connection ~ 8300 2600
+Wire Wire Line
+	8300 2600 8200 2600
+Wire Wire Line
+	8400 2800 8400 2250
+Wire Wire Line
+	8400 2250 3050 2250
+Wire Wire Line
+	3050 2250 3050 2800
+Wire Wire Line
+	5050 3500 5050 3600
+Wire Wire Line
+	5050 3600 6300 3600
+Wire Wire Line
+	6300 3600 6300 2500
+Wire Wire Line
+	7150 2650 8200 2650
+Connection ~ 7150 2650
+Connection ~ 8200 2650
+Wire Wire Line
+	8200 2650 8200 2800
+Wire Wire Line
+	6300 2500 7250 2500
+Wire Wire Line
+	7250 2500 7250 2800
 $EndSCHEMATC

Commit message: Layout for 65C816 CPU board
Parts:
- U3: footprint (none) -> Package_DIP:DIP-14_W7.62mm_Socket
Changed lines of the file:
@@
 	5050 2750 5050 2800
 Wire Wire Line
-	5050 2750 5550 2750
-Wire Wire Line
 	5550 2800 5550 2750
-Connection ~ 5550 2750
-Wire Wire Line
-	5550 2750 5650 2750
-Wire Wire Line
-	5650 2800 5650 2750
-Connection ~ 5650 2750
-Wire Wire Line
-	5650 2750 5750 2750
-Wire Wire Line
-	5750 2800 5750 2750
-Connection ~ 5750 2750
-Wire Wire Line
-	5750 2750 5850 2750
 Wire Wire Line
 	5850 2800 5850 2750
-Connection ~ 5850 2750
-Wire Wire Line
-	5850 2750 5950 2750
 Wire Wire Line
 	5950 2800 5950 2750
@@
 F 0 "U3" H 6650 3150 50  0000 R CNN
 F 1 "74AC00" V 6550 2900 50  0000 R CNN
-F 2 "" H 6550 3150 50  0001 C CNN
+F 2 "Package_DIP:DIP-14_W7.62mm_Socket" H 6550 3150 50  0001 C CNN
 F 3 "" H 6550 3150 50  0001 C CNN
 	1    6550 3150
@@
 Wire Wire Line
 	7250 2500 7250 2800
+Wire Wire Line
+	5650 2750 5750 2750
+Wire Wire Line
+	5850 2750 5950 2750
+Wire Wire Line
+	5750 2750 5850 2750
+Connection ~ 5850 2750
+Wire Wire Line
+	5750 2800 5750 2750
+Connection ~ 5750 2750
+Wire Wire Line
+	5650 2800 5650 2750
+Connection ~ 5650 2750
+Wire Wire Line
+	5550 2750 5650 2750
+Wire Wire Line
+	5050 2750 5550 2750
+Connection ~ 5550 2750
 $EndSCHEMATC

Commit message: Better layout for 65c816 CPU board
Connections:
- wire segments 188 -> 190
Changed lines of the file:
@@
 	6100 3250 6100 3550
 Wire Wire Line
-	5950 3550 6100 3550
+	5950 3550 6050 3550
 Connection ~ 6100 3550
 Wire Wire Line
@@
 Wire Wire Line
 	5050 2750 5050 2800
-Wire Wire Line
-	5550 2800 5550 2750
-Wire Wire Line
-	5850 2800 5850 2750
 Wire Wire Line
 	5950 2800 5950 2750
@@
 	7250 2500 7250 2800
 Wire Wire Line
-	5650 2750 5750 2750
-Wire Wire Line
-	5850 2750 5950 2750
-Wire Wire Line
-	5750 2750 5850 2750
-Connection ~ 5850 2750
-Wire Wire Line
-	5750 2800 5750 2750
-Connection ~ 5750 2750
-Wire Wire Line
-	5650 2800 5650 2750
-Connection ~ 5650 2750
-Wire Wire Line
-	5550 2750 5650 2750
-Wire Wire Line
-	5050 2750 5550 2750
-Connection ~ 5550 2750
+	5050 2750 5950 2750
+Wire Wire Line
+	5550 2800 5550 2650
+Wire Wire Line
+	6050 2650 6050 3550
+Wire Wire Line
+	5550 2650 5650 2650
+Connection ~ 6050 3550
+Wire Wire Line
+	6050 3550 6100 3550
+Wire Wire Line
+	5650 2800 5650 2650
+Connection ~ 5650 2650
+Wire Wire Line
+	5650 2650 5750 2650
+Wire Wire Line
+	5750 2800 5750 2650
+Connection ~ 5750 2650
+Wire Wire Line
+	5750 2650 5850 2650
+Wire Wire Line
+	5850 2800 5850 2650
+Connection ~ 5850 2650
+Wire Wire Line
+	5850 2650 6050 2650
 $EndSCHEMATC
