File: mainboard/mainboard.sch (KiCad schematic (older format))
At the start: 77 parts, among them U1 74HC04, U2 AS6C4008, U3 74HC32, U4 74HC00, U5 SST39SF040, U6 NE555, U7 74HCT245, U8 74HC574, U9 74HC574, Y1 Crystal

Commit message: Main board layout tweaks
Parts:
- C3, C5: value 22pF -> 47pF
Connections:
- net labels added: OERAM, OEROM, RDIN, WROUT, XX
Changed lines of the file:
@@
 P 1750 7100
 F 0 "C3" H 1842 7146 50  0000 L CNN
-F 1 "22pF" H 1842 7055 50  0000 L CNN
+F 1 "47pF" H 1842 7055 50  0000 L CNN
 F 2 "Capacitor_THT:C_Disc_D5.0mm_W2.5mm_P5.00mm" H 1750 7100 50  0001 C CNN
 F 3 "~" H 1750 7100 50  0001 C CNN
@@
 P 2350 7100
 F 0 "C5" H 2442 7146 50  0000 L CNN
-F 1 "22pF" H 2442 7055 50  0000 L CNN
+F 1 "47pF" H 2442 7055 50  0000 L CNN
 F 2 "Capacitor_THT:C_Disc_D5.0mm_W2.5mm_P5.00mm" H 2350 7100 50  0001 C CNN
 F 3 "~" H 2350 7100 50  0001 C CNN
@@
 	2900 1100 2900 900
 $Comp
-L power:+5V #PWR?
+L power:+5V #PWR0102
 U 1 1 5F01DB81
 P 2900 850
-F 0 "#PWR?" H 2900 700 50  0001 C CNN
+F 0 "#PWR0102" H 2900 700 50  0001 C CNN
 F 1 "+5V" H 2915 1023 50  0000 C CNN
 F 2 "" H 2900 850 50  0001 C CNN
@@
 	2900 850  2900 900
 Connection ~ 2900 900
+Text Label 7550 4050 0    50   ~ 0
+WROUT
+Text Label 7900 2150 0    50   ~ 0
+RDIN
+Text Label 3200 2300 0    50   ~ 0
+OERAM
+Text Label 5400 2300 0    50   ~ 0
+OEROM
+Text Label 7200 2050 0    50   ~ 0
+XX
 $EndSCHEMATC

Commit message: More PCB design First tiny program running
Parts:
- removed C12: 100nF, Capacitor_THT:C_Disc_D3.8mm_W2.6mm_P2.50mm, symbol Device:C_Small
- removed D1, D2, D3, D4, D5, D6, D7, D8: LED_Small, LED_THT:LED_D3.0mm, symbol Device:LED_Small
- removed JOUT2: Conn_01x08_Male, Connector_PinHeader_2.54mm:PinHeader_1x08_P2.54mm_Vertical, symbol Connector:Conn_01x08_Male
- removed R12, R13, R14, R15, R16, R17, R18, R19: 1k, Resistor_THT:R_Axial_DIN0207_L6.3mm_D2.5mm_P7.62mm_Horizontal, symbol Device:R_Small
- removed STANDOFF1, STANDOFF2, STANDOFF3, STANDOFF4: Conn_01x01_Male, Connector_PinHeader_2.54mm:PinHeader_1x01_P2.54mm_Vertical, symbol Connector:Conn_01x01_Male
- removed U8: 74HC574, Package_DIP:DIP-20_W7.62mm_Socket, symbol 74xx:74HCT574
- R10, R11, R4, R5, R6, R7, R8, R9: value 10k -> 22k
- U3: value 74HC32 -> 74AC32
- U4: value 74HC00 -> 74AC00
- U7: value 74HCT245 -> 74HC245
- renumbered D16 to D0, D15 to D1, D14 to D2, D13 to D3, D12 to D4, D11 to D5, D10 to D6, D9 to D7
Connections:
- wire segments 397 -> 325
- no-connect marks 11 -> 8
Other:
- moved on the sheet: U1C, U1D, U1E, U1F, U4B, U7, U9

Commit message: Repurposing this repo (and product name) for my gernic 8-bit computer main board.
Parts:
- removed JIN1, JOUT1: Conn_01x08_Male, Connector_PinHeader_2.54mm:PinHeader_1x08_P2.54mm_Vertical, symbol Connector:Conn_01x08_Male
- removed JIOPOWER1: Conn_01x02_Male, Connector_PinHeader_2.54mm:PinHeader_1x02_P2.54mm_Vertical, symbol Connector:Conn_01x02_Male
- removed R10, R11, R5, R6, R7, R8, R9: 22k, Resistor_THT:R_Axial_DIN0207_L6.3mm_D2.5mm_P7.62mm_Horizontal, symbol Device:R_Small
- removed R20, R21, R22, R23, R24, R25, R26, R27: 1k, Resistor_THT:R_Axial_DIN0207_L6.3mm_D2.5mm_P7.62mm_Horizontal, symbol Device:R_Small
- removed SWRESET1: SW_Push, Button_Switch_THT:SW_PUSH_6mm, symbol Switch:SW_Push
- added D9: LED_Small, LED_THT:LED_D3.0mm, symbol Device:LED_Small
- added JIN1, JOUT1: Conn_01x08_Female, Connector_PinSocket_2.54mm:PinSocket_1x08_P2.54mm_Vertical, symbol Connector:Conn_01x08_Female
- added JIOPOWER1: Conn_01x02_Female, Connector_PinSocket_2.54mm:PinSocket_1x02_P2.54mm_Vertical, symbol Connector:Conn_01x02_Female
- added RN1: 22k, Resistor_THT:R_Array_SIP9, symbol Device:R_Network08
- added RN2, RN3: 1k, Resistor_THT:R_Array_SIP8, symbol Device:R_Pack04_SIP
- added RN4: 1k, Resistor_THT:R_Array_SIP9, symbol Device:R_Network08
- added SW1: SW_DPDT_x2, Button_Switch_THT:SW_CuK_JS202011CQN_DPDT_Straight, symbol Switch:SW_DPDT_x2
- R3: value 470k -> 1M
- R4: value 22k -> 1k
Connections:
- net labels added: CERAM
- net labels removed: A19N
- wire segments 325 -> 339
- no-connect marks 8 -> 9
Other:
- moved on the sheet: U1C, U1F, U4A

Commit message: Redesign port access to use a state flip-flop made of NANDs instead of wasting a bit of the dedicatd output IC.
Parts:
- C3, C5: value 47pF -> 33pF
- U1: value 74HC04 -> 74AC04
Connections:
- net labels added: CPOUTPUT, IOMODE, OEINPUT, RESETIO
- net labels removed: RAM_INHIBIT, RDIN, WROUT, XX
- wire segments 339 -> 347
- no-connect marks 9 -> 5
Other:
- note added: "CLOCK"
- note added: "INPUT"
- note added: "MODE\nREGISTER"
- note added: "OUTPUT"
- note added: "POWER-ON RESET"
- moved on the sheet: U1A, U1B, U1C, U1D, U1E, U1F, U1G, U4A, U4B, U4C, U4D, U4E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

Commit message: Rename A19 to RAM to create two distinct address spaces.
Parts:
- U1: value 74AC04 -> 74HC04
Connections:
- net labels added: RAM
- net labels removed: A19
Changed lines of the file:
@@
 A18
 Text Label 1200 2250 0    50   ~ 0
-A19
+RAM
 $Comp
 L power:GND #PWR04
@@
 $EndComp
 Text Label 2100 1900 0    50   ~ 0
-A19
+RAM
 Text Label 3000 1900 0    50   ~ 0
 CERAM
@@
 RD
 Text Label 4100 2550 0    50   ~ 0
-A19
+RAM
 Wire Wire Line
 	4100 2350 4450 2350
@@
 WR
 Text Label 6250 1900 0    50   ~ 0
-A19
+RAM
 Wire Wire Line
 	6250 1700 6500 1700
@@
 IOMODE
 Text Label 5200 1050 0    50   ~ 0
-A19
+RAM
 Wire Wire Line
 	5200 850  5750 850
@@
 P 2150 5900
 F 0 "U1" H 2150 6217 50  0000 C CNN
-F 1 "74AC04" H 2150 6126 50  0000 C CNN
+F 1 "74HC04" H 2150 6126 50  0000 C CNN
 F 2 "Package_DIP:DIP-14_W7.62mm_Socket" H 2150 5900 50  0001 C CNN
 F 3 "http://www.nxp.com/documents/data_sheet/74HC_HCT04.pdf" H 2150 5900 50  0001 C CNN
@@
 P 1150 6750
 F 0 "U1" H 1380 6796 50  0000 L CNN
-F 1 "74AC04" H 1380 6705 50  0000 L CNN
+F 1 "74HC04" H 1380 6705 50  0000 L CNN
 F 2 "Package_DIP:DIP-14_W7.62mm_Socket" H 1150 6750 50  0001 C CNN
 F 3 "http://www.nxp.com/documents/data_sheet/74HC_HCT04.pdf" H 1150 6750 50  0001 C CNN
@@
 P 2850 5900
 F 0 "U1" H 2850 6217 50  0000 C CNN
-F 1 "74AC04" H 2850 6126 50  0000 C CNN
+F 1 "74HC04" H 2850 6126 50  0000 C CNN
 F 2 "Package_DIP:DIP-14_W7.62mm_Socket" H 2850 5900 50  0001 C CNN
 F 3 "http://www.nxp.com/documents/data_sheet/74HC_HCT04.pdf" H 2850 5900 50  0001 C CNN
@@
 P 3500 5900
 F 0 "U1" H 3500 6217 50  0000 C CNN
-F 1 "74AC04" H 3500 6126 50  0000 C CNN
+F 1 "74HC04" H 3500 6126 50  0000 C CNN
 F 2 "Package_DIP:DIP-14_W7.62mm_Socket" H 3500 5900 50  0001 C CNN
 F 3 "http://www.nxp.com/documents/data_sheet/74HC_HCT04.pdf" H 3500 5900 50  0001 C CNN
@@
 P 6050 6150
 F 0 "U1" H 6050 6467 50  0000 C CNN
-F 1 "74AC04" H 6050 6376 50  0000 C CNN
+F 1 "74HC04" H 6050 6376 50  0000 C CNN
 F 2 "Package_DIP:DIP-14_W7.62mm_Socket" H 6050 6150 50  0001 C CNN
 F 3 "http://www.nxp.com/documents/data_sheet/74HC_HCT04.pdf" H 6050 6150 50  0001 C CNN
@@
 P 2600 1900
 F 0 "U1" H 2600 2217 50  0000 C CNN
-F 1 "74AC04" H 2600 2126 50  0000 C CNN
+F 1 "74HC04" H 2600 2126 50  0000 C CNN
 F 2 "Package_DIP:DIP-14_W7.62mm_Socket" H 2600 1900 50  0001 C CNN
 F 3 "http://www.nxp.com/documents/data_sheet/74HC_HCT04.pdf" H 2600 1900 50  0001 C CNN
@@
 P 4350 1550
 F 0 "U1" H 4350 1867 50  0000 C CNN
-F 1 "74AC04" H 4350 1776 50  0000 C CNN
+F 1 "74HC04" H 4350 1776 50  0000 C CNN
 F 2 "Package_DIP:DIP-14_W7.62mm_Socket" H 4350 1550 50  0001 C CNN
 F 3 "http://www.nxp.com/documents/data_sheet/74HC_HCT04.pdf" H 4350 1550 50  0001 C CNN
@@
 	4650 1550 4750 1550
 Text Label 4450 1750 0    50   ~ 0
-A19
+RAM
 Wire Wire Line
 	4450 1750 4750 1750

Commit message: Switch meaning of the A19 pin from RAM to ROM. Use pull-ups instead of pull-downs for the input port.
Parts:
- RN1: value 22k -> 10k
Connections:
- net labels added: RD#, RES#, ROM, WR#
- net labels removed: CERAM, RD, RES, WR
Changed lines of the file:
@@
 A18
 Text Label 1200 2250 0    50   ~ 0
-RAM
+ROM
 $Comp
 L power:GND #PWR04
@@
 CLK
 Text Label 1200 1950 0    50   ~ 0
-RES
+RES#
 Text Label 1200 2050 0    50   ~ 0
-WR
+WR#
 Text Label 1200 2150 0    50   ~ 0
-RD
+RD#
 Wire Wire Line
 	1150 1650 1200 1650
@@
 $EndComp
 Text Label 2100 1900 0    50   ~ 0
+ROM
+Text Label 3000 1900 0    50   ~ 0
 RAM
-Text Label 3000 1900 0    50   ~ 0
-CERAM
 $Comp
 L 74xx:74LS32 U3
@@
 $EndComp
 Text Label 3350 3700 0    50   ~ 0
-WR
+WR#
 Text Label 1950 2400 0    50   ~ 0
-RD
+RD#
 Text Label 1950 2600 0    50   ~ 0
 IOMODE
@@
 Connection ~ 5450 3400
 Text Label 4100 2350 0    50   ~ 0
-RD
+RD#
 Text Label 4100 2550 0    50   ~ 0
 RAM
@@
 	7800 5000 7950 5000
 $Comp
-L power:GND #PWR042
-U 1 1 5F00B794
-P 10750 2800
-F 0 "#PWR042" H 10750 2550 50  0001 C CNN
-F 1 "GND" H 10755 2627 50  0000 C CNN
-F 2 "" H 10750 2800 50  0001 C CNN
-F 3 "" H 10750 2800 50  0001 C CNN
-	1    10750 2800
-	-1   0    0    1
-$EndComp
-$Comp
 L power:GND #PWR035
 U 1 1 5F03240F
@@
 	9050 2000 9100 2000
 Text Label 6250 1700 0    50   ~ 0
-WR
+WR#
 Text Label 6250 1900 0    50   ~ 0
 RAM
@@
 	7600 3850 7950 3850
 Text Label 6300 1150 0    50   ~ 0
-RD
+RD#
 Wire Wire Line
 	6300 1150 6500 1150
@@
 $EndComp
 Text Label 6450 6150 0    50   ~ 0
-RES
+RES#
 Wire Wire Line
 	6350 6150 6450 6150
@@
 P 10550 3250
 F 0 "RN1" V 9950 3250 50  0000 C CNN
-F 1 "22k" V 10050 3250 50  0000 C CNN
+F 1 "10k" V 10050 3250 50  0000 C CNN
 F 2 "Resistor_THT:R_Array_SIP9" V 11025 3250 50  0001 C CNN
 F 3 "http://www.vishay.com/docs/31509/csc.pdf" H 10550 3250 50  0001 C CNN
@@
 	9800 1000 10000 1000
 Wire Wire Line
-	10750 2800 10750 2850
-Wire Wire Line
 	9800 1000 9800 1300
 Wire Wire Line
@@
 NoConn ~ 9400 1400
 Text Label 3350 4400 0    50   ~ 0
-CERAM
+ROM
 Text Label 3350 4200 0    50   ~ 0
 OERAM
@@
 	6000 4600 6400 4600
 Text Label 3850 1550 0    50   ~ 0
-WR
+WR#
 Wire Wire Line
 	3850 1550 4050 1550
@@
 Text Notes 4750 5450 0    79   ~ 0
 POWER-ON RESET
+$Comp
+L power:+5V #PWR?
+U 1 1 5EF0C22D
+P 10750 2750
+F 0 "#PWR?" H 10750 2600 50  0001 C CNN
+F 1 "+5V" H 10765 2923 50  0000 C CNN
+F 2 "" H 10750 2750 50  0001 C CNN
+F 3 "" H 10750 2750 50  0001 C CNN
+	1    10750 2750
+	1    0    0    -1
+$EndComp
+Wire Wire Line
+	10750 2750 10750 2850
 $EndSCHEMATC

Commit message: Add power input on pin header to allow USB device to drive the machine.
Parts:
- removed JIN1, JOUT1: Conn_01x08_Female, Connector_PinSocket_2.54mm:PinSocket_1x08_P2.54mm_Vertical, symbol Connector:Conn_01x08_Female
- removed JIOPOWER1: Conn_01x02_Female, Connector_PinSocket_2.54mm:PinSocket_1x02_P2.54mm_Vertical, symbol Connector:Conn_01x02_Female
- added JIN1, JOUT1: Conn_01x08_Male, Connector_PinHeader_2.54mm:PinHeader_1x08_P2.54mm_Vertical, symbol Connector:Conn_01x08_Male
- added JPOWER2: Conn_01x04_Male, Connector_PinHeader_2.54mm:PinHeader_1x04_P2.54mm_Vertical, symbol Connector:Conn_01x04_Male
Connections:
- net labels added: VIN
- wire segments 347 -> 349
Changed lines of the file:
@@
 L power:GND #PWR043
 U 1 1 5F619573
-P 9050 1900
-F 0 "#PWR043" H 9050 1650 50  0001 C CNN
-F 1 "GND" V 9055 1772 50  0000 R CNN
-F 2 "" H 9050 1900 50  0001 C CNN
-F 3 "" H 9050 1900 50  0001 C CNN
-	1    9050 1900
+P 9800 2100
+F 0 "#PWR043" H 9800 1850 50  0001 C CNN
+F 1 "GND" V 9805 1972 50  0000 R CNN
+F 2 "" H 9800 2100 50  0001 C CNN
+F 3 "" H 9800 2100 50  0001 C CNN
+	1    9800 2100
 	0    1    1    0
 $EndComp
@@
 L power:+5V #PWR044
 U 1 1 5F61965F
-P 9050 2000
-F 0 "#PWR044" H 9050 1850 50  0001 C CNN
-F 1 "+5V" V 9065 2128 50  0000 L CNN
-F 2 "" H 9050 2000 50  0001 C CNN
-F 3 "" H 9050 2000 50  0001 C CNN
-	1    9050 2000
+P 9800 2200
+F 0 "#PWR044" H 9800 2050 50  0001 C CNN
+F 1 "+5V" V 9815 2328 50  0000 L CNN
+F 2 "" H 9800 2200 50  0001 C CNN
+F 3 "" H 9800 2200 50  0001 C CNN
+	1    9800 2200
 	0    -1   -1   0
 $EndComp
 Wire Wire Line
-	9050 1900 9100 1900
-Wire Wire Line
-	9050 2000 9100 2000
+	9800 2100 9850 2100
+Wire Wire Line
+	9800 2200 9850 2200
 Text Label 6250 1700 0    50   ~ 0
 WR#
@@
 L Connector:Barrel_Jack_Switch JPOWER1
 U 1 1 610F8C76
-P 10300 1100
-F 0 "JPOWER1" H 10355 1417 50  0000 C CNN
-F 1 "Barrel_Jack_Switch" H 10355 1326 50  0000 C CNN
-F 2 "Connector_BarrelJack:BarrelJack_Horizontal" H 10350 1060 50  0001 C CNN
-F 3 "~" H 10350 1060 50  0001 C CNN
-	1    10300 1100
+P 10500 1100
+F 0 "JPOWER1" H 10555 1417 50  0000 C CNN
+F 1 "Barrel_Jack_Switch" H 10555 1326 50  0000 C CNN
+F 2 "Connector_BarrelJack:BarrelJack_Horizontal" H 10550 1060 50  0001 C CNN
+F 3 "~" H 10550 1060 50  0001 C CNN
+	1    10500 1100
 	-1   0    0    -1
 $EndComp
@@
 	3150 5900 3200 5900
 Wire Wire Line
-	10000 1100 9950 1100
+	10200 1100 9950 1100
 Wire Wire Line
 	9950 1100 9950 1200
 Wire Wire Line
-	9950 1200 10000 1200
+	9950 1200 10200 1200
 $Comp
 L Device:R_Small R4
@@
 Wire Wire Line
 	9000 3750 9550 3750
-$Comp
-L Connector:Conn_01x02_Female JIOPOWER1
-U 1 1 5F57B80C
-P 9300 1900
-F 0 "JIOPOWER1" H 9327 1876 50  0000 L CNN
-F 1 "Conn_01x02_Female" H 9327 1785 50  0000 L CNN
-F 2 "Connector_PinSocket_2.54mm:PinSocket_1x02_P2.54mm_Vertical" H 9300 1900 50  0001 C CNN
-F 3 "~" H 9300 1900 50  0001 C CNN
-	1    9300 1900
-	1    0    0    -1
-$EndComp
-$Comp
-L Connector:Conn_01x08_Female JIN1
-U 1 1 5F57DA6E
-P 10300 3100
-F 0 "JIN1" H 10193 2475 50  0000 C CNN
-F 1 "Conn_01x08_Female" H 10250 2550 50  0000 C CNN
-F 2 "Connector_PinSocket_2.54mm:PinSocket_1x08_P2.54mm_Vertical" H 10300 3100 50  0001 C CNN
-F 3 "~" H 10300 3100 50  0001 C CNN
-	1    10300 3100
-	1    0    0    -1
-$EndComp
-Connection ~ 10100 3300
-Connection ~ 10100 3200
-Connection ~ 10100 3100
-Connection ~ 10100 3000
-Connection ~ 10100 2900
-Connection ~ 10100 2800
-$Comp
-L Connector:Conn_01x08_Female JOUT1
-U 1 1 5F5A8239
-P 9250 5300
-F 0 "JOUT1" H 9143 4675 50  0000 C CNN
-F 1 "Conn_01x08_Female" H 9200 4750 50  0000 C CNN
-F 2 "Connector_PinSocket_2.54mm:PinSocket_1x08_P2.54mm_Vertical" H 9250 5300 50  0001 C CNN
-F 3 "~" H 9250 5300 50  0001 C CNN
-	1    9250 5300
-	1    0    0    -1
-$EndComp
 Wire Wire Line
 	9150 3400 9950 3400
@@
 L power:GND #PWR0103
 U 1 1 5F60ACC5
-P 9950 1350
-F 0 "#PWR0103" H 9950 1100 50  0001 C CNN
-F 1 "GND" H 9955 1177 50  0000 C CNN
-F 2 "" H 9950 1350 50  0001 C CNN
-F 3 "" H 9950 1350 50  0001 C CNN
-	1    9950 1350
-	1    0    0    -1
-$EndComp
-Wire Wire Line
-	9950 1200 9950 1350
+P 9950 1250
+F 0 "#PWR0103" H 9950 1000 50  0001 C CNN
+F 1 "GND" H 9955 1077 50  0000 C CNN
+F 2 "" H 9950 1250 50  0001 C CNN
+F 3 "" H 9950 1250 50  0001 C CNN
+	1    9950 1250
+	1    0    0    -1
+$EndComp
+Wire Wire Line
+	9950 1200 9950 1250
 Connection ~ 9800 1000
 Wire Wire Line
-	9800 1000 10000 1000
+	9800 1000 10200 1000
 Wire Wire Line
 	9800 1000 9800 1300
@@
 POWER-ON RESET
 $Comp
-L power:+5V #PWR?
+L power:+5V #PWR0101
 U 1 1 5EF0C22D
 P 10750 2750
-F 0 "#PWR?" H 10750 2600 50  0001 C CNN
+F 0 "#PWR0101" H 10750 2600 50  0001 C CNN
 F 1 "+5V" H 10765 2923 50  0000 C CNN
 F 2 "" H 10750 2750 50  0001 C CNN
@@
 Wire Wire Line
 	10750 2750 10750 2850
+$Comp
+L Connector:Conn_01x04_Male JPOWER2
+U 1 1 5EF2E021
+P 10050 2000
+F 0 "JPOWER2" H 10023 1973 50  0000 R CNN
+F 1 "Conn_01x04_Male" H 10023 1882 50  0000 R CNN
+F 2 "Connector_PinHeader_2.54mm:PinHeader_1x04_P2.54mm_Vertical" H 10050 2000 50  0001 C CNN
+F 3 "~" H 10050 2000 50  0001 C CNN
+	1    10050 2000
+	-1   0    0    -1
+$EndComp
+$Comp
+L power:GND #PWR0102
+U 1 1 5EF2EE7D
+P 9800 2000
+F 0 "#PWR0102" H 9800 1750 50  0001 C CNN
+F 1 "GND" V 9805 1872 50  0000 R CNN
+F 2 "" H 9800 2000 50  0001 C CNN
+F 3 "" H 9800 2000 50  0001 C CNN
+	1    9800 2000
+	0    1    1    0
+$EndComp
+Wire Wire Line
+	9800 2000 9850 2000
+Text Label 9550 1900 0    50   ~ 0
+VIN
+Wire Wire Line
+	9550 1900 9850 1900
+Text Label 9900 1000 0    50   ~ 0
+VIN
+$Comp
+L Connector:Conn_01x08_Male JIN1
+U 1 1 5EFDCCD8
+P 10300 3100
+F 0 "JIN1" H 10450 2550 50  0000 R CNN
+F 1 "Conn_01x08_Male" H 10450 2450 50  0000 R CNN
+F 2 "Connector_PinHeader_2.54mm:PinHeader_1x08_P2.54mm_Vertical" H 10300 3100 50  0001 C CNN
+F 3 "~" H 10300 3100 50  0001 C CNN
+	1    10300 3100
+	-1   0    0    -1
+$EndComp
+Connection ~ 10100 2800
+Connection ~ 10100 2900
+Connection ~ 10100 3000
+Connection ~ 10100 3100
+Connection ~ 10100 3200
+Connection ~ 10100 3300
+$Comp
+L Connector:Conn_01x08_Male JOUT1
+U 1 1 5EFDE82B
+P 9250 5300
+F 0 "JOUT1" H 9400 4750 50  0000 R CNN
+F 1 "Conn_01x08_Male" H 9400 4650 50  0000 R CNN
+F 2 "Connector_PinHeader_2.54mm:PinHeader_1x08_P2.54mm_Vertical" H 9250 5300 50  0001 C CNN
+F 3 "~" H 9250 5300 50  0001 C CNN
+	1    9250 5300
+	-1   0    0    -1
+$EndComp
 $EndSCHEMATC
