File: mainboard/mainboard.sch (KiCad schematic (older format))
At the start: 44 parts, among them SW1 SW_DPDT_x2, U1 74HC04, U2 AS6C4008, U3 74AC32, U4 74AC00, U5 SST39SF040, U6 NE555, U7 74HC245, U9 74HC574, Y1 Crystal

Commit message: Remove protection resistors for input port. Stagger ports so an IO board will have better mechanical stability
Parts:
- removed RN2, RN3: 1k, Resistor_THT:R_Array_SIP8, symbol Device:R_Pack04_SIP
Connections:
- wire segments 349 -> 311
Changed lines of the file:
@@
 L Device:R_Network08 RN1
 U 1 1 5F268690
-P 10550 3250
-F 0 "RN1" V 9950 3250 50  0000 C CNN
-F 1 "10k" V 10050 3250 50  0000 C CNN
-F 2 "Resistor_THT:R_Array_SIP9" V 11025 3250 50  0001 C CNN
-F 3 "http://www.vishay.com/docs/31509/csc.pdf" H 10550 3250 50  0001 C CNN
-	1    10550 3250
+P 9800 3200
+F 0 "RN1" V 9200 3200 50  0000 C CNN
+F 1 "10k" V 9300 3200 50  0000 C CNN
+F 2 "Resistor_THT:R_Array_SIP9" V 10275 3200 50  0001 C CNN
+F 3 "http://www.vishay.com/docs/31509/csc.pdf" H 9800 3200 50  0001 C CNN
+	1    9800 3200
 	0    1    1    0
 $EndComp
-$Comp
-L Device:R_Pack04_SIP RN3
-U 1 1 5F0C3E00
-P 9350 3150
-F 0 "RN3" V 8650 3150 50  0000 L CNN
-F 1 "1k" V 8750 3150 50  0000 L CNN
-F 2 "Resistor_THT:R_Array_SIP8" V 10025 3150 50  0001 C CNN
-F 3 "http://www.vishay.com/docs/31509/csc.pdf" H 9350 3150 50  0001 C CNN
-	1    9350 3150
-	0    1    1    0
-$EndComp
-$Comp
-L Device:R_Pack04_SIP RN2
-U 1 1 5F1112A9
-P 9750 3350
-F 0 "RN2" V 9050 3350 50  0000 L CNN
-F 1 "1k" V 9150 3350 50  0000 L CNN
-F 2 "Resistor_THT:R_Array_SIP8" V 10425 3350 50  0001 C CNN
-F 3 "http://www.vishay.com/docs/31509/csc.pdf" H 9750 3350 50  0001 C CNN
-	1    9750 3350
-	0    1    1    0
-$EndComp
-Wire Wire Line
-	9150 2750 9150 2800
-Wire Wire Line
-	9150 3050 9150 3100
-Wire Wire Line
-	9150 3100 10000 3100
-Wire Wire Line
-	9150 3350 9150 3400
-Wire Wire Line
-	9150 3650 9150 3700
-Wire Wire Line
-	9150 2800 10100 2800
-Wire Wire Line
-	10000 3100 10000 3000
-Wire Wire Line
-	10000 3000 10100 3000
-Wire Wire Line
-	9550 2950 9550 3000
-Wire Wire Line
-	9550 3000 9950 3000
-Wire Wire Line
-	9950 3000 9950 2900
-Wire Wire Line
-	9950 2900 10100 2900
-Wire Wire Line
-	10100 3100 10050 3100
-Wire Wire Line
-	10050 3100 10050 3150
-Wire Wire Line
-	9550 3300 9550 3250
-Wire Wire Line
-	9950 3400 9950 3350
-Wire Wire Line
-	9950 3350 10000 3350
-Wire Wire Line
-	9950 3300 9950 3150
-Wire Wire Line
-	9950 3150 10050 3150
-Wire Wire Line
-	10000 3350 10000 3200
-Wire Wire Line
-	10000 3200 10100 3200
-Wire Wire Line
-	9550 3550 9550 3600
-Wire Wire Line
-	10000 3600 10000 3400
-Wire Wire Line
-	10000 3400 10050 3400
-Wire Wire Line
-	10050 3300 10100 3300
-Wire Wire Line
-	10050 3700 10050 3450
-Wire Wire Line
-	10050 3450 10100 3450
-Wire Wire Line
-	10100 3450 10100 3400
-Wire Wire Line
-	9550 3850 9550 3900
-Wire Wire Line
-	10100 3900 10100 3550
-Wire Wire Line
-	10100 3450 10350 3450
-Connection ~ 10100 3450
-Wire Wire Line
-	10100 3550 10350 3550
-Connection ~ 10100 3550
-Wire Wire Line
-	10100 3550 10100 3500
-Wire Wire Line
-	10100 3200 10100 3250
-Wire Wire Line
-	10100 3250 10350 3250
-Wire Wire Line
-	10100 3300 10100 3350
-Wire Wire Line
-	10100 3350 10350 3350
-Wire Wire Line
-	10050 3300 10050 3400
-Wire Wire Line
-	10100 3100 10100 3150
-Wire Wire Line
-	10100 3150 10350 3150
-Wire Wire Line
-	10100 3000 10100 3050
-Wire Wire Line
-	10100 3050 10350 3050
-Wire Wire Line
-	10100 2900 10100 2950
-Wire Wire Line
-	10100 2950 10350 2950
-Wire Wire Line
-	10100 2800 10100 2850
-Wire Wire Line
-	10100 2850 10350 2850
-Wire Wire Line
-	8950 2850 8950 2650
-Wire Wire Line
-	8950 2650 9150 2650
-Wire Wire Line
-	8950 2950 9000 2950
-Wire Wire Line
-	9000 2950 9000 2850
-Wire Wire Line
-	9000 2850 9550 2850
-Wire Wire Line
-	9050 2950 9150 2950
-Wire Wire Line
-	8950 3150 9550 3150
-Wire Wire Line
-	8950 3250 9150 3250
-Wire Wire Line
-	8950 3050 9050 3050
-Wire Wire Line
-	9050 2950 9050 3050
-Wire Wire Line
-	8950 3350 9100 3350
-Wire Wire Line
-	9100 3350 9100 3450
-Wire Wire Line
-	9100 3450 9550 3450
-Wire Wire Line
-	8950 3450 9050 3450
-Wire Wire Line
-	9050 3450 9050 3550
-Wire Wire Line
-	9050 3550 9150 3550
-Wire Wire Line
-	8950 3550 9000 3550
-Wire Wire Line
-	9000 3550 9000 3750
-Wire Wire Line
-	9000 3750 9550 3750
-Wire Wire Line
-	9150 3400 9950 3400
-Wire Wire Line
-	9550 3300 9950 3300
-Wire Wire Line
-	9550 3600 10000 3600
-Wire Wire Line
-	9150 3700 10050 3700
-Wire Wire Line
-	9550 3900 10100 3900
-$Comp
-L Switch:SW_DPDT_x2 SW1
-U 1 1 5F5ED49A
-P 9600 1000
-F 0 "SW1" H 9600 1285 50  0000 C CNN
-F 1 "SW_DPDT_x2" H 9600 1194 50  0000 C CNN
-F 2 "Button_Switch_THT:SW_CuK_JS202011CQN_DPDT_Straight" H 9600 1000 50  0001 C CNN
-F 3 "" H 9600 1000 50  0001 C CNN
-	1    9600 1000
-	-1   0    0    -1
-$EndComp
-$Comp
-L Switch:SW_DPDT_x2 SW1
-U 2 1 5F5ED53F
-P 9600 1300
-F 0 "SW1" H 9600 1100 50  0000 C CNN
-F 1 "SW_DPDT_x2" H 9600 1000 50  0000 C CNN
-F 2 "Button_Switch_THT:SW_CuK_JS202011CQN_DPDT_Straight" H 9600 1300 50  0001 C CNN
-F 3 "" H 9600 1300 50  0001 C CNN
-	2    9600 1300
-	-1   0    0    -1
-$EndComp
+Wire Wire Line
+	8950 3050 9000 3050
 $Comp
 L power:GND #PWR0103
@@
 Wire Wire Line
 	9950 1200 9950 1250
-Connection ~ 9800 1000
 Wire Wire Line
 	9800 1000 10200 1000
@@
 L power:+5V #PWR0101
 U 1 1 5EF0C22D
-P 10750 2750
-F 0 "#PWR0101" H 10750 2600 50  0001 C CNN
-F 1 "+5V" H 10765 2923 50  0000 C CNN
-F 2 "" H 10750 2750 50  0001 C CNN
-F 3 "" H 10750 2750 50  0001 C CNN
-	1    10750 2750
+P 10000 2750
+F 0 "#PWR0101" H 10000 2600 50  0001 C CNN
+F 1 "+5V" H 10015 2923 50  0000 C CNN
+F 2 "" H 10000 2750 50  0001 C CNN
+F 3 "" H 10000 2750 50  0001 C CNN
+	1    10000 2750
 	1    0    0    -1
 $EndComp
-Wire Wire Line
-	10750 2750 10750 2850
 $Comp
 L Connector:Conn_01x04_Male JPOWER2
@@
 L Connector:Conn_01x08_Male JIN1
 U 1 1 5EFDCCD8
-P 10300 3100
-F 0 "JIN1" H 10450 2550 50  0000 R CNN
-F 1 "Conn_01x08_Male" H 10450 2450 50  0000 R CNN
-F 2 "Connector_PinHeader_2.54mm:PinHeader_1x08_P2.54mm_Vertical" H 10300 3100 50  0001 C CNN
-F 3 "~" H 10300 3100 50  0001 C CNN
-	1    10300 3100
-	-1   0    0    -1
-$EndComp
-Connection ~ 10100 2800
-Connection ~ 10100 2900
-Connection ~ 10100 3000
-Connection ~ 10100 3100
-Connection ~ 10100 3200
-Connection ~ 10100 3300
+P 9250 3150
+F 0 "JIN1" H 9400 2600 50  0000 R CNN
+F 1 "Conn_01x08_Male" H 9400 2500 50  0000 R CNN
+F 2 "Connector_PinHeader_2.54mm:PinHeader_1x08_P2.54mm_Vertical" H 9250 3150 50  0001 C CNN
+F 3 "~" H 9250 3150 50  0001 C CNN
+	1    9250 3150
+	-1   0    0    -1
+$EndComp
 $Comp
 L Connector:Conn_01x08_Male JOUT1
@@
 	-1   0    0    -1
 $EndComp
+Wire Wire Line
+	8950 2850 9000 2850
+Wire Wire Line
+	8950 2950 9000 2950
+Wire Wire Line
+	8950 3150 9000 3150
+Wire Wire Line
+	8950 3250 9000 3250
+Wire Wire Line
+	8950 3350 9000 3350
+Wire Wire Line
+	8950 3550 9000 3550
+Wire Wire Line
+	10000 2800 10000 2750
+Wire Wire Line
+	9000 2850 9000 2800
+Wire Wire Line
+	9000 2800 9600 2800
+Connection ~ 9000 2850
+Wire Wire Line
+	9000 2850 9050 2850
+Wire Wire Line
+	9000 2950 9000 2900
+Wire Wire Line
+	9000 2900 9600 2900
+Connection ~ 9000 2950
+Wire Wire Line
+	9000 2950 9050 2950
+Wire Wire Line
+	9000 3050 9000 3000
+Wire Wire Line
+	9000 3000 9600 3000
+Connection ~ 9000 3050
+Wire Wire Line
+	9000 3050 9050 3050
+Wire Wire Line
+	9000 3150 9000 3100
+Wire Wire Line
+	9000 3100 9600 3100
+Connection ~ 9000 3150
+Wire Wire Line
+	9000 3150 9050 3150
+Wire Wire Line
+	9000 3250 9000 3200
+Wire Wire Line
+	9000 3200 9600 3200
+Connection ~ 9000 3250
+Wire Wire Line
+	9000 3250 9050 3250
+Wire Wire Line
+	9000 3350 9000 3300
+Wire Wire Line
+	9000 3300 9600 3300
+Connection ~ 9000 3350
+Wire Wire Line
+	9000 3350 9050 3350
+Wire Wire Line
+	8950 3450 9000 3450
+Wire Wire Line
+	9000 3450 9000 3400
+Wire Wire Line
+	9000 3400 9600 3400
+Connection ~ 9000 3450
+Wire Wire Line
+	9000 3450 9050 3450
+Wire Wire Line
+	9000 3550 9000 3500
+Wire Wire Line
+	9000 3500 9600 3500
+Connection ~ 9000 3550
+Wire Wire Line
+	9000 3550 9050 3550
+$Comp
+L Switch:SW_DPDT_x2 SW1
+U 2 1 5F5ED53F
+P 9600 1300
+F 0 "SW1" H 9600 1100 50  0000 C CNN
+F 1 "SW_DPDT_x2" H 9600 1000 50  0000 C CNN
+F 2 "Button_Switch_THT:SW_CuK_JS202011CQN_DPDT_Straight" H 9600 1300 50  0001 C CNN
+F 3 "" H 9600 1300 50  0001 C CNN
+	2    9600 1300
+	-1   0    0    -1
+$EndComp
+Connection ~ 9800 1000
+$Comp
+L Switch:SW_DPDT_x2 SW1
+U 1 1 5F5ED49A
+P 9600 1000
+F 0 "SW1" H 9600 1285 50  0000 C CNN
+F 1 "SW_DPDT_x2" H 9600 1194 50  0000 C CNN
+F 2 "Button_Switch_THT:SW_CuK_JS202011CQN_DPDT_Straight" H 9600 1000 50  0001 C CNN
+F 3 "" H 9600 1000 50  0001 C CNN
+	1    9600 1000
+	-1   0    0    -1
+$EndComp
