File: mainboard/mainboard.sch (KiCad schematic (older format))
At the start: 42 parts, among them SW1 SW_DPDT_x2, U1 74HC04, U2 AS6C4008, U3 74AC32, U4 74AC00, U5 SST39SF040, U6 NE555, U7 74HC245, U9 74HC574, Y1 Crystal

Commit message: doc
Parts:
- SW1: footprint Button_Switch_THT:SW_CuK_JS202011CQN_DPDT_Straight -> ProjectFootprints:DPDS Switch
Changed lines of the file:
@@
 F 0 "SW1" H 9600 1100 50  0000 C CNN
 F 1 "SW_DPDT_x2" H 9600 1000 50  0000 C CNN
-F 2 "Button_Switch_THT:SW_CuK_JS202011CQN_DPDT_Straight" H 9600 1300 50  0001 C CNN
+F 2 "ProjectFootprints:DPDS Switch" H 9600 1300 50  0001 C CNN
 F 3 "" H 9600 1300 50  0001 C CNN
 	2    9600 1300
@@
 F 0 "SW1" H 9600 1285 50  0000 C CNN
 F 1 "SW_DPDT_x2" H 9600 1194 50  0000 C CNN
-F 2 "Button_Switch_THT:SW_CuK_JS202011CQN_DPDT_Straight" H 9600 1000 50  0001 C CNN
+F 2 "ProjectFootprints:DPDS Switch" H 9600 1000 50  0001 C CNN
 F 3 "" H 9600 1000 50  0001 C CNN
 	1    9600 1000

Commit message: Change mainboard to have larger holes for the ZIF socket and the power switch.
Parts:
- U5: footprint Package_DIP:DIP-32_W15.24mm_Socket -> ProjectFootprints:DIP-32_LargeHoles
Changed lines of the file:
@@
 Title "Byte machine - main board"
 Date ""
-Rev "1.0"
+Rev "2"
 Comp ""
 Comment1 ""
@@
 F 0 "U5" H 4850 6067 50  0000 C CNN
 F 1 "SST39SF040" H 4850 5976 50  0000 C CNN
-F 2 "Package_DIP:DIP-32_W15.24mm_Socket" H 4900 4100 50  0001 L CNN
+F 2 "ProjectFootprints:DIP-32_LargeHoles" H 4900 4100 50  0001 L CNN
 F 3 "http://download.intel.com/design/archives/flash/docs/29045101.pdf" H 4850 4850 50  0001 C CNN
 	1    4850 4600
