File: i8088/i8088board/i8088board.sch (KiCad schematic (older format))
At the start: 4 parts

Commit message: Circuit and test program for the Intel 8088
Parts:
- added C1, C2, C3: 100nF, symbol Device:C_Small
- added Q1: Q_NPN_CBE, symbol Device:Q_NPN_CBE
- added R1, R2: 10k, symbol Device:R_Small
- U2, U3: renamed from U?; value 74HC573 -> 74AC573
- gave numbers to parts that had none: 2
Connections:
- wire segments 16 -> 191
- no-connect marks 0 -> 10
