File: ByteCPU/cpuboard/registers.sch (KiCad schematic (older format))
At the start: 13 parts

Commit message: Fix mistake in SELPC signal generation. More docu.
Connections:
- net labels added: REGC0, REGC1, WRC#
- net labels removed: WRA#
- wire segments 285 -> 281
Changed lines of the file:
@@
 $EndComp
-Wire Wire Line
-	1000 2100 1350 2100
 Wire Wire Line
 	3350 2100 3350 1800
-Wire Wire Line
-	1000 2200 1250 2200
 Wire Wire Line
 	3450 2200 3450 1800
@@
 	10450 3900 10450 3500
 Connection ~ 8100 3900
-Connection ~ 1350 2100
-Wire Wire Line
-	1350 2100 3350 2100
-Connection ~ 1250 2200
-Wire Wire Line
-	1250 2200 3450 2200
 Wire Wire Line
 	2150 5250 1000 5250
@@
 Wire Wire Line
 	1000 5450 2350 5450
-Wire Wire Line
-	1250 2200 1250 6800
-Wire Wire Line
-	1350 2100 1350 6700
 Text Label 2150 4150 1    50   ~ 0
 R00
@@
 $EndComp
 Wire Wire Line
-	1700 6800 1250 6800
-Wire Wire Line
-	1350 6700 1700 6700
-Wire Wire Line
 	2700 6800 3250 6800
 Wire Wire Line
@@
 	950  7000 1700 7000
 Text HLabel 950  7000 0    50   Input ~ 0
-WRA#
+WRC#
 Text HLabel 1000 6100 0    50   Input ~ 0
 CLK
@@
 Text HLabel 9650 2450 1    50   Input ~ 0
 B7
+Text HLabel 950  6700 0    50   Input ~ 0
+REGC0
+Text HLabel 950  6800 0    50   Input ~ 0
+REGC1
+Wire Wire Line
+	1000 2200 3450 2200
+Wire Wire Line
+	1000 2100 3350 2100
+Wire Wire Line
+	950  6700 1700 6700
+Wire Wire Line
+	950  6800 1700 6800
 $EndSCHEMATC

Commit message: Re-arrange the interconnect to better match the pin layout of the various chips.
Parts:
- renumbered UA3 to UA0, UA2 to UA1, UA1 to UA2, UA0 to UA3, UB3 to UB0, UB2 to UB1, UB1 to UB2, UB0 to UB3, UR3 to UR0, UR2 to UR1, UR1 to UR2, UR0 to UR3
Connections:
- wire segments 281 -> 282

Commit message: Modifications to fit the wiring to the physical layout of the 7400 logic. Bugfix: RD line was active during JMP instruction.
Parts:
- renumbered UADEC1 to UDEC2
Changed lines of the file:
@@
 	1950 3550 1950 3500
 $Comp
-L 74xx:74LS139 UADEC1
+L 74xx:74LS139 UDEC2
 U 2 1 604930AC
 P 4900 7200
-F 0 "UADEC1" H 4900 7567 50  0000 C CNN
+F 0 "UDEC2" H 4900 7567 50  0000 C CNN
 F 1 "74HC139" H 4900 7476 50  0000 C CNN
 F 2 "" H 4900 7200 50  0001 C CNN
@@
 $EndComp
 $Comp
-L 74xx:74LS139 UADEC1
+L 74xx:74LS139 UDEC2
 U 3 1 6049310F
 P 6150 7200
-F 0 "UADEC1" V 5783 7200 50  0000 C CNN
+F 0 "UDEC2" V 5783 7200 50  0000 C CNN
 F 1 "74HC139" V 5874 7200 50  0000 C CNN
 F 2 "" H 6150 7200 50  0001 C CNN
@@
 	6650 7200 6650 7150
 $Comp
-L 74xx:74LS139 UADEC1
+L 74xx:74LS139 UDEC2
 U 1 1 6058657D
 P 2200 6800
-F 0 "UADEC1" H 2200 7167 50  0000 C CNN
+F 0 "UDEC2" H 2200 7167 50  0000 C CNN
 F 1 "74HC139" H 2200 7076 50  0000 C CNN
 F 2 "" H 2200 6800 50  0001 C CNN
@@
 	9200 5200 9200 5550
 $Comp
-L power:+5V #PWR?
+L power:+5V #PWR0143
 U 1 1 5FCDFD1A
 P 4350 7050
-F 0 "#PWR?" H 4350 6900 50  0001 C CNN
+F 0 "#PWR0143" H 4350 6900 50  0001 C CNN
 F 1 "+5V" H 4365 7223 50  0000 C CNN
 F 2 "" H 4350 7050 50  0001 C CNN
