File: ByteCPU/cpuboard/ALU.sch (KiCad schematic (older format))
At the start: 4 parts

Commit message: Re-arrange the interconnect to better match the pin layout of the various chips.
Connections:
- wire segments 146 -> 154

Commit message: Rework all opcodes to speed up the decoding stage by 10 ns
Connections:
- net labels added: SELMEM
- net labels removed: SELALU#
Changed lines of the file:
@@
 OP2
 Text HLabel 1250 6450 0    50   Input ~ 0
-SELALU#
+SELMEM
 Text HLabel 6100 6000 3    50   Input ~ 0
 D0
