File: ByteCPU/cpuboard/Addressing.sch (KiCad schematic (older format))
At the start: 10 parts, among them U1 7400

Commit message: Rework all opcodes to speed up the decoding stage by 10 ns
Parts:
- removed U1: 7400, symbol 74xx:7400
Connections:
- net labels added: SELADR
- net labels removed: SELPC
- wire segments 244 -> 230
Changed lines of the file:
@@
 	4300 1200 4300 1250
-$Comp
-L 74xx:74LS163 UCTR3
-U 1 1 5F8BBB76
-P 3650 3300
-F 0 "UCTR3" V 4100 3050 50  0000 R CNN
-F 1 "74HC163" V 4000 3050 50  0000 R CNN
-F 2 "" H 3650 3300 50  0001 C CNN
-F 3 "http://www.ti.com/lit/gpn/sn74LS163" H 3650 3300 50  0001 C CNN
-	1    3650 3300
-	0    -1   -1   0
-$EndComp
 $Comp
 L 74xx:74LS163 UCTR2
@@
 	3450 2800 3450 2400
 Wire Wire Line
-	3450 2400 2550 2400
-Wire Wire Line
-	2550 2400 2550 1750
-Wire Wire Line
 	3350 2800 3350 2500
 Wire Wire Line
@@
 	5200 2800 5200 2350
 Wire Wire Line
-	5200 2350 4700 2350
-Wire Wire Line
 	5000 2800 5000 2550
 Wire Wire Line
@@
 	8250 2800 8250 2350
 Wire Wire Line
-	8250 2350 7350 2350
-Wire Wire Line
 	8150 2800 8150 2450
 Wire Wire Line
@@
 Wire Wire Line
 	10000 2800 10000 2350
-Wire Wire Line
-	10000 2350 9500 2350
-Wire Wire Line
-	9900 2800 9900 2450
 Wire Wire Line
 	9800 2800 9800 2550
@@
 	3450 3800 3450 5400
 Connection ~ 3450 5400
-Wire Wire Line
-	2450 1750 2450 2300
-Wire Wire Line
-	2750 1750 2750 2150
-Wire Wire Line
-	3450 1750 3450 2300
 Wire Wire Line
 	6550 4700 6550 1950
@@
 $EndComp
 Wire Wire Line
-	9400 1750 9400 2100
-Wire Wire Line
-	9500 1750 9500 2350
-Wire Wire Line
-	9700 1750 9700 1950
-Wire Wire Line
-	10100 1750 10100 2450
-Wire Wire Line
-	10400 1750 10400 2550
-Wire Wire Line
 	10600 1750 10600 1850
 Wire Wire Line
 	8450 1750 8450 1850
 Wire Wire Line
-	8250 1750 8250 2250
-Wire Wire Line
-	7950 1750 7950 2450
-Wire Wire Line
-	7550 1750 7550 2150
-Wire Wire Line
-	7350 1750 7350 2350
-Wire Wire Line
-	7250 1750 7250 5400
-Wire Wire Line
 	5800 1750 5800 1850
-Wire Wire Line
-	5600 1750 5600 2550
-Wire Wire Line
-	5300 1750 5300 2450
-Wire Wire Line
-	5000 1750 5000 2450
-Wire Wire Line
-	4900 1750 4900 1950
-Wire Wire Line
-	4700 1750 4700 2350
 Wire Wire Line
 	3750 1750 3800 1750
@@
 D7
 Text HLabel 850  1850 0    50   Input ~ 0
-SELPC
+SELADR
 Wire Wire Line
 	3650 3800 3650 5700
@@
 	10300 3800 10300 5600
 Wire Wire Line
-	9800 1750 9800 2450
-Wire Wire Line
-	9800 2450 9700 2450
-Wire Wire Line
-	9700 2450 9700 2800
-Wire Wire Line
-	9900 2450 10100 2450
-Wire Wire Line
-	9800 2550 10400 2550
-Wire Wire Line
-	7950 2650 7650 2650
-Wire Wire Line
-	7650 1750 7650 2650
-Wire Wire Line
-	8150 2450 7950 2450
-Wire Wire Line
-	8050 2250 8250 2250
+	9800 2550 10300 2550
+Wire Wire Line
+	8050 2250 8150 2250
 Wire Wire Line
 	8050 2250 8050 2800
 Wire Wire Line
-	4900 2450 5000 2450
-Wire Wire Line
-	4900 2450 4900 2800
-Wire Wire Line
-	5100 2800 5100 2450
-Wire Wire Line
-	5100 2450 5300 2450
-Wire Wire Line
-	5000 2550 5600 2550
-Wire Wire Line
-	3150 2700 2850 2700
-Wire Wire Line
-	2850 1750 2850 2700
-Wire Wire Line
-	3250 2300 3450 2300
+	5000 2550 5500 2550
+Wire Wire Line
+	3250 2300 3350 2300
 Wire Wire Line
 	3250 2300 3250 2800
-Wire Wire Line
-	3350 2500 3150 2500
-Wire Wire Line
-	3150 2500 3150 1750
 Wire Wire Line
 	850  4700 1800 4700
@@
 	1400 5400 3450 5400
 Wire Wire Line
-	4900 1950 1800 1950
-Wire Wire Line
 	1800 1950 1800 2800
 Wire Wire Line
-	5500 2000 1900 2000
-Wire Wire Line
 	1900 2000 1900 2800
 Wire Wire Line
-	5500 1750 5500 2000
-Wire Wire Line
-	5200 1750 5200 2050
-Wire Wire Line
-	5200 2050 2000 2050
-Wire Wire Line
 	2000 2050 2000 2800
 Wire Wire Line
-	4600 1750 4600 2100
-Wire Wire Line
-	4600 2100 2100 2100
-Wire Wire Line
 	2100 2100 2100 2800
 Wire Wire Line
-	2750 2150 1700 2150
-Wire Wire Line
 	1700 2150 1700 2800
 Wire Wire Line
-	3350 2200 1600 2200
-Wire Wire Line
 	1600 2200 1600 2800
 Wire Wire Line
-	3350 1750 3350 2200
-Wire Wire Line
-	3050 1750 3050 2250
-Wire Wire Line
-	3050 2250 1500 2250
-Wire Wire Line
 	1500 2250 1500 2800
 Wire Wire Line
-	2450 2300 1400 2300
-Wire Wire Line
 	1400 2300 1400 2800
-Wire Wire Line
-	9700 1950 6550 1950
-Wire Wire Line
-	10000 1750 10000 2050
-Wire Wire Line
-	10300 2000 6650 2000
-Wire Wire Line
-	10300 1750 10300 2000
-Wire Wire Line
-	10000 2050 6750 2050
-Wire Wire Line
-	9400 2100 6850 2100
-Wire Wire Line
-	6950 2150 7550 2150
-Wire Wire Line
-	7850 2250 7150 2250
-Wire Wire Line
-	7850 1750 7850 2250
-Wire Wire Line
-	7050 2200 8150 2200
-Wire Wire Line
-	8150 1750 8150 2200
-Wire Wire Line
-	1050 5800 1750 5800
 Text HLabel 1050 5600 0    50   Input ~ 0
 COUNT
 Wire Wire Line
-	1050 5600 2000 5600
-Wire Wire Line
 	1050 5700 3650 5700
 Wire Wire Line
+	2550 2300 2550 1750
+Wire Wire Line
+	1400 2300 2550 2300
+Wire Wire Line
+	2450 1750 2450 2400
+Wire Wire Line
+	2450 2400 3450 2400
+Wire Wire Line
+	2850 2150 2850 1750
+Wire Wire Line
+	1700 2150 2850 2150
+Wire Wire Line
+	2750 2700 2750 1750
+Wire Wire Line
+	2750 2700 3150 2700
+Wire Wire Line
+	3150 2250 3150 1750
+Wire Wire Line
+	1500 2250 3150 2250
+Wire Wire Line
+	3050 1750 3050 2500
+Wire Wire Line
+	3050 2500 3350 2500
+Wire Wire Line
+	3450 2200 3450 1750
+Wire Wire Line
+	1600 2200 3450 2200
+Wire Wire Line
+	3350 1750 3350 2300
+Wire Wire Line
+	4700 2100 4700 1750
+Wire Wire Line
+	2100 2100 4700 2100
+Wire Wire Line
+	4600 1750 4600 2350
+Wire Wire Line
+	4600 2350 5200 2350
+Wire Wire Line
+	5000 1950 5000 1750
+Wire Wire Line
+	1800 1950 5000 1950
+Wire Wire Line
+	4900 1750 4900 2800
+Wire Wire Line
+	5300 2050 5300 1750
+Wire Wire Line
+	2000 2050 5300 2050
+Wire Wire Line
+	5200 1750 5200 2200
+Wire Wire Line
+	5600 2000 5600 1750
+Wire Wire Line
+	1900 2000 5600 2000
+Wire Wire Line
+	5500 1750 5500 2550
+Wire Wire Line
+	7250 2450 7350 2450
+Wire Wire Line
+	7350 2450 7350 1750
+Wire Wire Line
+	7250 2450 7250 5400
+Wire Wire Line
+	7250 1750 7250 2350
+Wire Wire Line
+	7250 2350 8250 2350
+Wire Wire Line
+	7650 2150 7650 1750
+Wire Wire Line
+	6950 2150 7650 2150
+Wire Wire Line
+	7550 1750 7550 2650
+Wire Wire Line
+	7550 2650 7950 2650
+Wire Wire Line
+	7950 2250 7950 1750
+Wire Wire Line
+	7150 2250 7950 2250
+Wire Wire Line
+	7850 1750 7850 2450
+Wire Wire Line
+	7850 2450 8150 2450
+Wire Wire Line
+	8250 2200 8250 1750
+Wire Wire Line
+	7050 2200 8250 2200
+Wire Wire Line
+	8150 1750 8150 2250
+Wire Wire Line
+	9500 2100 9500 1750
+Wire Wire Line
+	6850 2100 9500 2100
+Wire Wire Line
+	9400 1750 9400 2350
+Wire Wire Line
+	9400 2350 10000 2350
+Wire Wire Line
+	9800 1950 9800 1750
+Wire Wire Line
+	6550 1950 9800 1950
+Wire Wire Line
+	9700 1750 9700 2800
+Wire Wire Line
+	10100 2050 10100 1750
+Wire Wire Line
+	6750 2050 10100 2050
+Wire Wire Line
+	10000 1750 10000 2250
+Wire Wire Line
+	10400 2000 10400 1750
+Wire Wire Line
+	6650 2000 10400 2000
+Wire Wire Line
+	10300 1750 10300 2550
+Wire Wire Line
+	9900 2250 10000 2250
+Wire Wire Line
+	9900 2250 9900 2800
+Wire Wire Line
+	5100 2200 5200 2200
+Wire Wire Line
+	5100 2200 5100 2800
+Wire Wire Line
+	1050 5800 8450 5800
+$Comp
+L 74xx:74LS163 UCTR3
+U 1 1 5F8BBB76
+P 3650 3300
+F 0 "UCTR3" V 4100 3050 50  0000 R CNN
+F 1 "74HC163" V 4000 3050 50  0000 R CNN
+F 2 "" H 3650 3300 50  0001 C CNN
+F 3 "http://www.ti.com/lit/gpn/sn74LS163" H 3650 3300 50  0001 C CNN
+	1    3650 3300
+	0    -1   -1   0
+$EndComp
+Wire Wire Line
+	1050 5600 3750 5600
+Wire Wire Line
+	3750 3800 3750 5600
+Connection ~ 3750 5600
+Wire Wire Line
 	3750 5600 5500 5600
-$Comp
-L 74xx:7400 U?
-U 3 1 5FBA4C03
-P 2400 6400
-AR Path="/5FBA4C03" Ref="U?"  Part="3"
-AR Path="/60888F9A/5FBA4C03" Ref="U1"  Part="3"
-F 0 "U1" H 2400 6725 50  0000 C CNN
-F 1 "7400" H 2400 6634 50  0000 C CNN
-F 2 "" H 2400 6400 50  0001 C CNN
-F 3 "http://www.ti.com/lit/gpn/sn7400" H 2400 6400 50  0001 C CNN
-	3    2400 6400
-	1    0    0    -1
-$EndComp
-$Comp
-L 74xx:7400 U?
-U 4 1 5FBA4C16
-P 3150 6400
-AR Path="/5FBA4C16" Ref="U?"  Part="4"
-AR Path="/60888F9A/5FBA4C16" Ref="U1"  Part="4"
-F 0 "U1" H 3350 6650 50  0000 C CNN
-F 1 "7400" H 3350 6550 50  0000 C CNN
-F 2 "" H 3150 6400 50  0001 C CNN
-F 3 "http://www.ti.com/lit/gpn/sn7400" H 3150 6400 50  0001 C CNN
-	4    3150 6400
-	1    0    0    -1
-$EndComp
-Wire Wire Line
-	2100 6300 2000 6300
-Wire Wire Line
-	2000 6300 2000 5600
-Connection ~ 2000 5600
-Wire Wire Line
-	2000 5600 3750 5600
-Wire Wire Line
-	2100 6500 1750 6500
-Wire Wire Line
-	1750 6500 1750 5800
-Connection ~ 1750 5800
-Wire Wire Line
-	1750 5800 8450 5800
-Wire Wire Line
-	2750 6300 2850 6300
-Wire Wire Line
-	2750 6500 2850 6500
-Wire Wire Line
-	3750 6400 3450 6400
-Wire Wire Line
-	3750 3800 3750 6400
-Wire Wire Line
-	2750 6300 2750 6400
-Wire Wire Line
-	2700 6400 2750 6400
-Connection ~ 2750 6400
-Wire Wire Line
-	2750 6400 2750 6500
 $EndSCHEMATC
