File: ByteCPU/cpuboard/Control.sch (KiCad schematic (older format))
At the start: 8 parts, among them U1 74HC00, U2 74HC32, U3 74HC08, U4 74HC11, U5 74HC11

Commit message: Fix mistake in SELPC signal generation. More docu.
Connections:
- net labels added: WRC#
- net labels removed: WRA#
- wire segments 170 -> 171
Changed lines of the file:
@@
 L 74xx:74LS32 U2
 U 2 1 602800E1
-P 5250 4550
-F 0 "U2" H 5250 4875 50  0000 C CNN
-F 1 "74HC32" H 5250 4784 50  0000 C CNN
-F 2 "" H 5250 4550 50  0001 C CNN
-F 3 "http://www.ti.com/lit/gpn/sn74LS32" H 5250 4550 50  0001 C CNN
-	2    5250 4550
+P 10300 4150
+F 0 "U2" H 10300 4475 50  0000 C CNN
+F 1 "74HC32" H 10300 4384 50  0000 C CNN
+F 2 "" H 10300 4150 50  0001 C CNN
+F 3 "http://www.ti.com/lit/gpn/sn74LS32" H 10300 4150 50  0001 C CNN
+	2    10300 4150
 	1    0    0    -1
 $EndComp
@@
 	1950 5300 2250 5300
 Wire Wire Line
-	1950 5150 1950 5500
-Wire Wire Line
 	2250 5300 2550 5300
 Connection ~ 2250 5300
@@
 L 74xx:74LS08 U3
 U 4 1 6031320F
-P 10300 4150
-F 0 "U3" H 10300 4350 50  0000 C CNN
-F 1 "74HC08" H 10550 4300 50  0000 C CNN
-F 2 "" H 10300 4150 50  0001 C CNN
-F 3 "http://www.ti.com/lit/gpn/sn74LS08" H 10300 4150 50  0001 C CNN
-	4    10300 4150
+P 10300 5300
+F 0 "U3" H 10300 5500 50  0000 C CNN
+F 1 "74HC08" H 10550 5450 50  0000 C CNN
+F 2 "" H 10300 5300 50  0001 C CNN
+F 3 "http://www.ti.com/lit/gpn/sn74LS08" H 10300 5300 50  0001 C CNN
+	4    10300 5300
 	1    0    0    -1
 $EndComp
@@
 $EndComp
 Wire Wire Line
-	5550 3350 6450 3350
-Wire Wire Line
-	4950 3250 1950 3250
+	5550 3350 6100 3350
 Connection ~ 1950 3250
 Wire Wire Line
 	1950 3250 1950 4150
-Wire Wire Line
-	4950 3350 2050 3350
 Connection ~ 2050 3350
 Wire Wire Line
@@
 	1    0    0    -1
 $EndComp
-Wire Wire Line
-	4950 4650 4950 5200
-Connection ~ 4950 5200
-Wire Wire Line
-	4800 4450 4800 5500
-Wire Wire Line
-	4800 5500 1950 5500
-Wire Wire Line
-	4800 4450 4950 4450
-Connection ~ 1950 5500
-Wire Wire Line
-	5550 4550 6450 4550
 $Comp
 L 74xx:74HC00 U1
@@
 	4100 5400 6450 5400
 Connection ~ 4100 5400
-Text HLabel 6450 4550 2    50   Input ~ 0
+Text HLabel 6450 3500 2    50   Input ~ 0
 SELPC
 Text HLabel 6450 3350 2    50   Input ~ 0
@@
 SELALU#
 Text HLabel 6450 750  2    50   Input ~ 0
-WRA#
+WRC#
 Wire Wire Line
 	2050 750  2050 2050
@@
 L power:GND #PWR0206
 U 1 1 6108204C
-P 9950 4950
-F 0 "#PWR0206" H 9950 4700 50  0001 C CNN
-F 1 "GND" H 9955 4777 50  0000 C CNN
-F 2 "" H 9950 4950 50  0001 C CNN
-F 3 "" H 9950 4950 50  0001 C CNN
-	1    9950 4950
-	1    0    0    -1
-$EndComp
-Wire Wire Line
-	9950 4950 9950 4850
+P 9950 5450
+F 0 "#PWR0206" H 9950 5200 50  0001 C CNN
+F 1 "GND" H 9955 5277 50  0000 C CNN
+F 2 "" H 9950 5450 50  0001 C CNN
+F 3 "" H 9950 5450 50  0001 C CNN
+	1    9950 5450
+	1    0    0    -1
+$EndComp
 Connection ~ 9950 4850
 Text HLabel 3500 7400 3    50   Input ~ 0
@@
 	2150 5700 2150 5950
 Wire Wire Line
-	1950 5500 1950 5950
-Wire Wire Line
 	2050 5600 2050 5950
 $Comp
@@
 NoConn ~ 2450 4150
 NoConn ~ 2550 4150
+Wire Wire Line
+	1950 5150 1950 5950
+Wire Wire Line
+	6100 3350 6100 3500
+Wire Wire Line
+	6100 3500 6450 3500
+Connection ~ 6100 3350
+Wire Wire Line
+	6100 3350 6450 3350
+Wire Wire Line
+	1950 3250 4950 3250
+Wire Wire Line
+	2050 3350 4950 3350
+Wire Wire Line
+	9950 5200 10000 5200
+Wire Wire Line
+	9950 4850 9950 5200
+Wire Wire Line
+	9950 5200 9950 5400
+Wire Wire Line
+	9950 5400 10000 5400
+Connection ~ 9950 5200
+Wire Wire Line
+	9950 5400 9950 5450
+Connection ~ 9950 5400
 $EndSCHEMATC

Commit message: Share logic ICs between control and addressing to save 2 parts.
Parts:
- removed unit 4 of U1
- removed unit 4 of U2
- removed unit 4 of U3
Connections:
- wire segments 171 -> 159
- no-connect marks 6 -> 4
Changed lines of the file:
@@
 	4300 5200 2650 5200
-$Comp
-L 74xx:74LS32 U2
-U 2 1 602800E1
-P 10300 4150
-F 0 "U2" H 10300 4475 50  0000 C CNN
-F 1 "74HC32" H 10300 4384 50  0000 C CNN
-F 2 "" H 10300 4150 50  0001 C CNN
-F 3 "http://www.ti.com/lit/gpn/sn74LS32" H 10300 4150 50  0001 C CNN
-	2    10300 4150
-	1    0    0    -1
-$EndComp
 $Comp
 L 74xx:74HC00 U1
@@
 	1    0    0    -1
 $EndComp
-$Comp
-L 74xx:74LS08 U3
-U 4 1 6031320F
-P 10300 5300
-F 0 "U3" H 10300 5500 50  0000 C CNN
-F 1 "74HC08" H 10550 5450 50  0000 C CNN
-F 2 "" H 10300 5300 50  0001 C CNN
-F 3 "http://www.ti.com/lit/gpn/sn74LS08" H 10300 5300 50  0001 C CNN
-	4    10300 5300
-	1    0    0    -1
-$EndComp
 Wire Wire Line
 	5550 2900 6450 2900
@@
 L 74xx:74LS32 U2
 U 3 1 603435D4
-P 7500 1850
-F 0 "U2" H 7500 2175 50  0000 C CNN
-F 1 "74HC32" H 7500 2084 50  0000 C CNN
-F 2 "" H 7500 1850 50  0001 C CNN
-F 3 "http://www.ti.com/lit/gpn/sn74LS32" H 7500 1850 50  0001 C CNN
-	3    7500 1850
+P 7500 2350
+F 0 "U2" H 7500 2650 50  0000 C CNN
+F 1 "74HC32" H 7500 2550 50  0000 C CNN
+F 2 "" H 7500 2350 50  0001 C CNN
+F 3 "http://www.ti.com/lit/gpn/sn74LS32" H 7500 2350 50  0001 C CNN
+	3    7500 2350
 	1    0    0    -1
 $EndComp
@@
 $Comp
 L 74xx:74HC00 U1
-U 4 1 60354CFB
-P 10300 4750
-F 0 "U1" H 10400 4950 50  0000 R CNN
-F 1 "74HC00" H 10750 4900 50  0000 R CNN
-F 2 "" H 10300 4750 50  0001 C CNN
-F 3 "http://www.ti.com/lit/gpn/sn74hc00" H 10300 4750 50  0001 C CNN
-	4    10300 4750
-	1    0    0    -1
-$EndComp
-$Comp
-L 74xx:74HC00 U1
 U 5 1 60354D96
 P 9100 1350
@@
 F 3 "http://www.ti.com/lit/gpn/sn74LS08" H 10650 1350 50  0001 C CNN
 	5    10650 1350
-	1    0    0    -1
-$EndComp
-$Comp
-L 74xx:74LS32 U2
-U 4 1 603565C8
-P 7500 2350
-F 0 "U2" H 7500 2675 50  0000 C CNN
-F 1 "74HC32" H 7500 2584 50  0000 C CNN
-F 2 "" H 7500 2350 50  0001 C CNN
-F 3 "http://www.ti.com/lit/gpn/sn74LS32" H 7500 2350 50  0001 C CNN
-	4    7500 2350
 	1    0    0    -1
 $EndComp
@@
 Wire Wire Line
 	2550 6950 2600 6950
-NoConn ~ 10600 4150
-NoConn ~ 10600 4750
-Wire Wire Line
-	9950 4850 10000 4850
-Wire Wire Line
-	9950 4850 9950 4650
-Wire Wire Line
-	9950 4650 10000 4650
-Wire Wire Line
-	9950 4650 9950 4250
-Wire Wire Line
-	9950 4250 10000 4250
-Connection ~ 9950 4650
-Wire Wire Line
-	9950 4250 9950 4050
-Wire Wire Line
-	9950 4050 10000 4050
-Connection ~ 9950 4250
 Text HLabel 1550 7550 3    50   Input ~ 0
 D0
@@
 Wire Wire Line
 	2250 3800 4950 3800
-$Comp
-L power:GND #PWR0206
-U 1 1 6108204C
-P 9950 5450
-F 0 "#PWR0206" H 9950 5200 50  0001 C CNN
-F 1 "GND" H 9955 5277 50  0000 C CNN
-F 2 "" H 9950 5450 50  0001 C CNN
-F 3 "" H 9950 5450 50  0001 C CNN
-	1    9950 5450
-	1    0    0    -1
-$EndComp
-Connection ~ 9950 4850
 Text HLabel 3500 7400 3    50   Input ~ 0
 ISTRUE
@@
 Wire Wire Line
 	2050 3350 4950 3350
-Wire Wire Line
-	9950 5200 10000 5200
-Wire Wire Line
-	9950 4850 9950 5200
-Wire Wire Line
-	9950 5200 9950 5400
-Wire Wire Line
-	9950 5400 10000 5400
-Connection ~ 9950 5200
-Wire Wire Line
-	9950 5400 9950 5450
-Connection ~ 9950 5400
+$Comp
+L 74xx:74LS32 U2
+U 2 1 5F9AE1AE
+P 7500 1850
+AR Path="/6088908D/5F9AE1AE" Ref="U2"  Part="2"
+AR Path="/60888F9A/5F9AE1AE" Ref="U?"  Part="2"
+F 0 "U2" H 7500 2150 50  0000 C CNN
+F 1 "74HC32" H 7500 2050 50  0000 C CNN
+F 2 "" H 7500 1850 50  0001 C CNN
+F 3 "http://www.ti.com/lit/gpn/sn74LS32" H 7500 1850 50  0001 C CNN
+	2    7500 1850
+	1    0    0    -1
+$EndComp
 $EndSCHEMATC

Commit message: Modifications to fit the wiring to the physical layout of the 7400 logic. Bugfix: RD line was active during JMP instruction.
Parts:
- removed U4: 74HC11, symbol 74xx:74LS11
- added unit 4 of U2
- added unit 4 of U3
- added unit 4 of U4
- renumbered U1 to U4
Connections:
- net labels added: COUNT, LOADHIGH#, LOADLOW#
- net labels removed: PCOP0, PCOP1
- wire segments 159 -> 158
- no-connect marks 4 -> 6
Other:
- moved on the sheet: U4B, U4C, U4E, USTATE1A, USTATE1B

Commit message: Rework control logic to allow and additional IO instruction
Connections:
- net labels added: IO#, IOCMD#
- wire segments 158 -> 167
- no-connect marks 6 -> 3
Other:
- moved on the sheet: U4C

Commit message: Rework all opcodes to speed up the decoding stage by 10 ns
Connections:
- net labels added: ALU#, SELADR, SELMEM
- net labels removed: ALUOP#, IO#, IOCMD#, SELALU#, SELPC
- wire segments 167 -> 155
- no-connect marks 3 -> 4
Other:
- moved on the sheet: U4C, U4D
