File: IOexpander/ioexpanderboard/ioexpanderboard.sch (KiCad schematic (older format))
At the start: 12 parts, among them U1 ATtiny44-20PU, U2 74LVC245, U3 LD1117S33TR_SOT223

Commit message: Redefine ByteCPU to implement it in 7400 logic. Prototype of assembler.
Connections:
- wire segments 84 -> 81
- no-connect marks 19 -> 20
Changed lines of the file:
@@
 Text Label 1750 3100 0    50   ~ 0
 MISO
-Text Label 1750 3300 0    50   ~ 0
+Text Label 1750 3400 0    50   ~ 0
 RX2
 Wire Wire Line
@@
 Text Label 6100 2100 0    50   ~ 0
 RTS
-Text Label 6100 1700 0    50   ~ 0
+Text Label 6100 2600 0    50   ~ 0
 RX2
 Wire Wire Line
@@
 NoConn ~ 5950 2400
 NoConn ~ 5950 2500
-NoConn ~ 5950 2600
 Wire Wire Line
 	5950 2100 6100 2100
@@
 	6200 1500 6200 1300
 Wire Wire Line
-	1650 3300 1700 3300
-Wire Wire Line
-	5950 1700 6100 1700
-Wire Wire Line
 	5950 1900 6600 1900
 NoConn ~ 5950 2200
@@
 NoConn ~ 8450 4600
 NoConn ~ 8450 4500
-Wire Wire Line
-	1650 3400 1700 3400
-Wire Wire Line
-	1700 3400 1700 3300
-Connection ~ 1700 3300
-Wire Wire Line
-	1700 3300 1750 3300
 $Comp
 L power:+5V #PWR?
@@
 Wire Wire Line
 	1650 3200 1900 3200
+NoConn ~ 1650 3300
+Wire Wire Line
+	1650 3400 1750 3400
+Wire Wire Line
+	5950 2600 6100 2600
+NoConn ~ 5950 1700
 $EndSCHEMATC

Commit message: Production files for cpu board. More work on IO expander board
Parts:
- removed C1: 100nF, Capacitor_THT:C_Disc_D3.0mm_W2.0mm_P2.50mm, symbol Device:C_Small
- removed D1: 1N4148, Diode_THT:D_DO-35_SOD27_P7.62mm_Horizontal, symbol Diode:1N4148
- removed JIN1: Conn_01x04_Male, Connector_PinHeader_2.54mm:PinHeader_1x04_P2.54mm_Vertical, symbol Connector:Conn_01x04_Male
- removed JOUT1: Conn_01x05_Male, Connector_PinHeader_2.54mm:PinHeader_1x05_P2.54mm_Vertical, symbol Connector:Conn_01x05_Male
- removed JUART1: Conn_01x04_Male, Connector_PinHeader_2.54mm:PinHeader_1x04_P2.54mm_Horizontal, symbol Connector:Conn_01x04_Male
- removed U1: ATtiny44-20PU, Package_DIP:DIP-14_W7.62mm_LongPads, symbol MCU_Microchip_ATtiny:ATtiny44-20PU
- removed U2: 74LVC245, Package_DIP:DIP-20_W7.62mm_LongPads, symbol 74xx:74LS245
- added C2: 10uF, Capacitor_SMD:C_0805_2012Metric_Pad1.15x1.40mm_HandSolder, symbol Device:C_Small
- added JINPUT1, JOUTPUT1: Conn_01x08_Male, Connector_PinHeader_2.54mm:PinHeader_1x08_P2.54mm_Vertical, symbol Connector:Conn_01x08_Male
- added JSERIAL1, JSERIAL2: DB9_Male, Connector_Dsub:DSUB-9_Male_Horizontal_P2.77x2.54mm_EdgePinOffset9.40mm, symbol Connector:DB9_Male
- added R2, R3, R4: 330, Resistor_SMD:R_0805_2012Metric_Pad1.15x1.40mm_HandSolder, symbol Device:R_Small
- added U1: 74LVC86, Package_SO:SOIC-14_3.9x8.7mm_P1.27mm, symbol 74xx:74HC86
- C1: renamed from C2; footprint Capacitor_THT:C_Disc_D3.0mm_W2.0mm_P2.50mm -> Capacitor_SMD:C_0805_2012Metric_Pad1.15x1.40mm_HandSolder
- R1: value 10k -> 330; footprint Resistor_THT:R_Axial_DIN0207_L6.3mm_D2.5mm_P7.62mm_Horizontal -> Resistor_SMD:R_0805_2012Metric_Pad1.15x1.40mm_HandSolder
- renumbered JPOWER2 to JPOWER1, U3 to U2
Connections:
- net labels added: CARD_DETECT, CS, CTS1, CTS2, RTS1, RTS2, RXD1, RXD2, TXD1, TXD2, WRITE_PROTECT
- net labels removed: RTS, RX, RX2, SS, TX
- wire segments 81 -> 82
- no-connect marks 20 -> 12
Other:
- moved on the sheet: U2
